File: Lark/Flash.kicad_sch (KiCad schematic)
At the start: 2 parts, among them U15 W25Q128JVSIQ

Commit message: Update, WIP
- Added TVS diode to 24v Supply.
- Fixed bleeder circuit at some point (I think it was this commit)
- Added Jumper to connect NTC to ADC. (again I think it was this commit)
Parts:
- C45: now not fitted
Changed lines of the file:
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@@
 		(dnp no)
 		(fields_autoplaced yes)
-		(property "Reference" "#PWR0180"
+		(property "Reference" "#PWR0184"
 			(at 168.91 111.76 0)
 			(effects
@@
 			(project "Lark"
 				(path "/a351af57-4353-47da-9f45-7393de572768/510bbd44-ee11-40bc-952d-6cd0def4c817/fbf20d92-3dc5-48bd-8ff0-5e0b8683d6ab"
-					(reference "#PWR0180")
+					(reference "#PWR0184")
 					(unit 1)
 				)
@@
 		(dnp no)
 		(fields_autoplaced yes)
-		(property "Reference" "#PWR0179"
+		(property "Reference" "#PWR0183"
 			(at 168.91 86.36 0)
 			(effects
@@
 			(project "Lark"
 				(path "/a351af57-4353-47da-9f45-7393de572768/510bbd44-ee11-40bc-952d-6cd0def4c817/fbf20d92-3dc5-48bd-8ff0-5e0b8683d6ab"
-					(reference "#PWR0179")
+					(reference "#PWR0183")
 					(unit 1)
 				)
@@
 		(in_bom yes)
 		(on_board yes)
-		(dnp no)
+		(dnp yes)
 		(property "Reference" "C45"
 			(at 173.736 93.472 0)
