File: Lark/USB.kicad_sch (KiCad schematic)
At the start: 4 parts, among them J2 2169890002, U9 USBLC6-2SC6

Commit message: Update, WIP
- Added TVS diode to 24v Supply.
- Fixed bleeder circuit at some point (I think it was this commit)
- Added Jumper to connect NTC to ADC. (again I think it was this commit)
Parts:
- renumbered R36 to R39, R37 to R40
Changed lines of the file:
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@@
 		(dnp no)
 		(fields_autoplaced yes)
-		(property "Reference" "#PWR093"
+		(property "Reference" "#PWR097"
 			(at 57.15 87.63 0)
 			(effects
@@
 			(project ""
 				(path "/a351af57-4353-47da-9f45-7393de572768/9aa817d4-eb96-4675-9e22-be0e45d55bef"
-					(reference "#PWR093")
+					(reference "#PWR097")
 					(unit 1)
 				)
@@
 		(dnp no)
 		(fields_autoplaced yes)
-		(property "Reference" "#PWR092"
+		(property "Reference" "#PWR096"
 			(at 57.15 31.75 0)
 			(effects
@@
 			(project ""
 				(path "/a351af57-4353-47da-9f45-7393de572768/9aa817d4-eb96-4675-9e22-be0e45d55bef"
-					(reference "#PWR092")
+					(reference "#PWR096")
 					(unit 1)
 				)
@@
 		(dnp no)
 		(fields_autoplaced yes)
-		(property "Reference" "#PWR094"
+		(property "Reference" "#PWR098"
 			(at 147.32 121.92 0)
 			(effects
@@
 			(project "Lark"
 				(path "/a351af57-4353-47da-9f45-7393de572768/9aa817d4-eb96-4675-9e22-be0e45d55bef"
-					(reference "#PWR094")
+					(reference "#PWR098")
 					(unit 1)
 				)
@@
 		(on_board yes)
 		(dnp no)
-		(property "Reference" "R37"
+		(property "Reference" "R40"
 			(at 41.91 120.6499 0)
 			(effects
@@
 			(project "Lark"
 				(path "/a351af57-4353-47da-9f45-7393de572768/9aa817d4-eb96-4675-9e22-be0e45d55bef"
-					(reference "R37")
+					(reference "R40")
 					(unit 1)
 				)
@@
 		(on_board yes)
 		(dnp no)
-		(property "Reference" "R36"
+		(property "Reference" "R39"
 			(at 27.94 120.6499 0)
 			(effects
@@
 			(project "Lark"
 				(path "/a351af57-4353-47da-9f45-7393de572768/9aa817d4-eb96-4675-9e22-be0e45d55bef"
-					(reference "R36")
+					(reference "R39")
 					(unit 1)
 				)
@@
 		(dnp no)
 		(fields_autoplaced yes)
-		(property "Reference" "#PWR095"
+		(property "Reference" "#PWR099"
 			(at 99.06 129.54 0)
 			(effects
@@
 			(project "Lark"
 				(path "/a351af57-4353-47da-9f45-7393de572768/9aa817d4-eb96-4675-9e22-be0e45d55bef"
-					(reference "#PWR095")
+					(reference "#PWR099")
 					(unit 1)
 				)
@@
 		(dnp no)
 		(fields_autoplaced yes)
-		(property "Reference" "#PWR096"
+		(property "Reference" "#PWR0100"
 			(at 25.4 139.7 0)
 			(effects
@@
 			(project "Lark"
 				(path "/a351af57-4353-47da-9f45-7393de572768/9aa817d4-eb96-4675-9e22-be0e45d55bef"
-					(reference "#PWR096")
+					(reference "#PWR0100")
 					(unit 1)
 				)
@@
 		(dnp no)
 		(fields_autoplaced yes)
-		(property "Reference" "#PWR097"
+		(property "Reference" "#PWR0101"
 			(at 39.37 139.7 0)
 			(effects
@@
 			(project "Lark"
 				(path "/a351af57-4353-47da-9f45-7393de572768/9aa817d4-eb96-4675-9e22-be0e45d55bef"
-					(reference "#PWR097")
-					(unit 1)
-				)
+					(reference "#PWR0101")
+					(unit 1)
+				)

Commit message: updated WIP
- fixed high-side switch (swapped out pfets)
- swapped out bleeder fet.
- changed a few footprints.
- changed zeners to 15v ones
- added soft-start cap back in to the high-side switch.

(today ive mainly been struggling with the inrush current, but I think its solved now)
Parts:
- renumbered U9 to U11
Changed lines of the file:
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@@
+		(dnp no)
+		(fields_autoplaced yes)
+		(property "Reference" "#PWR098"
+			(at 57.15 87.63 0)
+			(effects
+				(font
+					(size 1.27 1.27)
+				)
+				(hide yes)
+			)
+		)
+		(property "Value" "GND"
+			(at 57.15 86.36 0)
+			(effects
+				(font
+					(size 1.27 1.27)
+				)
+			)
+		)
+		(property "Footprint" ""
+			(at 57.15 81.28 0)
+			(effects
+				(font
+					(size 1.27 1.27)
+				)
+				(hide yes)
+			)
+		)
+		(property "Datasheet" ""
+			(at 57.15 81.28 0)
+			(effects
+				(font
+					(size 1.27 1.27)
+				)
+				(hide yes)
+			)
+		)
+		(property "Description" "Power symbol creates a global label with name \"GND\" , ground"
+			(at 57.15 81.28 0)
+			(effects
+				(font
+					(size 1.27 1.27)
+				)
+				(hide yes)
+			)
+		)
+		(pin "1"
+		)
+		(instances
+			(project ""
+				(path "/a351af57-4353-47da-9f45-7393de572768/9aa817d4-eb96-4675-9e22-be0e45d55bef"
+					(reference "#PWR098")
+					(unit 1)
+				)
+			)
+		)
+	)
+	(symbol
+		(lib_id "power:+5V")
+		(at 57.15 27.94 0)
+		(unit 1)
+		(exclude_from_sim no)
+		(in_bom yes)
+		(on_board yes)
 		(dnp no)
 		(fields_autoplaced yes)
 		(property "Reference" "#PWR097"
-			(at 57.15 87.63 0)
-			(effects
-				(font
-					(size 1.27 1.27)
-				)
-				(hide yes)
-			)
-		)
-		(property "Value" "GND"
-			(at 57.15 86.36 0)
-			(effects
-				(font
-					(size 1.27 1.27)
-				)
-			)
-		)
-		(property "Footprint" ""
-			(at 57.15 81.28 0)
-			(effects
-				(font
-					(size 1.27 1.27)
-				)
-				(hide yes)
-			)
-		)
-		(property "Datasheet" ""
-			(at 57.15 81.28 0)
-			(effects
-				(font
-					(size 1.27 1.27)
-				)
-				(hide yes)
-			)
-		)
-		(property "Description" "Power symbol creates a global label with name \"GND\" , ground"
-			(at 57.15 81.28 0)
-			(effects
-				(font
-					(size 1.27 1.27)
-				)
-				(hide yes)
-			)
-		)
-		(pin "1"
-		)
-		(instances
-			(project ""
-				(path "/a351af57-4353-47da-9f45-7393de572768/9aa817d4-eb96-4675-9e22-be0e45d55bef"
-					(reference "#PWR097")
-					(unit 1)
-				)
-			)
-		)
-	)
-	(symbol
-		(lib_id "power:+5V")
-		(at 57.15 27.94 0)
-		(unit 1)
-		(exclude_from_sim no)
-		(in_bom yes)
-		(on_board yes)
-		(dnp no)
-		(fields_autoplaced yes)
-		(property "Reference" "#PWR096"
 			(at 57.15 31.75 0)
 			(effects
@@
 			(project ""
 				(path "/a351af57-4353-47da-9f45-7393de572768/9aa817d4-eb96-4675-9e22-be0e45d55bef"
-					(reference "#PWR096")
+					(reference "#PWR097")
 					(unit 1)
 				)
@@
 		(dnp no)
 		(fields_autoplaced yes)
-		(property "Reference" "#PWR098"
+		(property "Reference" "#PWR099"
 			(at 147.32 121.92 0)
 			(effects
@@
 			(project "Lark"
 				(path "/a351af57-4353-47da-9f45-7393de572768/9aa817d4-eb96-4675-9e22-be0e45d55bef"
-					(reference "#PWR098")
+					(reference "#PWR099")
 					(unit 1)
 				)
@@
 		(on_board yes)
 		(dnp no)
-		(property "Reference" "U9"
+		(property "Reference" "U11"
 			(at 109.22 103.886 0)
 			(effects
@@
 			(project ""
 				(path "/a351af57-4353-47da-9f45-7393de572768/9aa817d4-eb96-4675-9e22-be0e45d55bef"
-					(reference "U9")
+					(reference "U11")
 					(unit 1)
 				)
@@
 		(dnp no)
 		(fields_autoplaced yes)
-		(property "Reference" "#PWR099"
+		(property "Reference" "#PWR0100"
 			(at 99.06 129.54 0)
 			(effects
@@
 			(project "Lark"
 				(path "/a351af57-4353-47da-9f45-7393de572768/9aa817d4-eb96-4675-9e22-be0e45d55bef"
-					(reference "#PWR099")
+					(reference "#PWR0100")
 					(unit 1)
 				)
@@
 		(dnp no)
 		(fields_autoplaced yes)
-		(property "Reference" "#PWR0100"
+		(property "Reference" "#PWR0101"
 			(at 25.4 139.7 0)
 			(effects
@@
 			(project "Lark"
 				(path "/a351af57-4353-47da-9f45-7393de572768/9aa817d4-eb96-4675-9e22-be0e45d55bef"
-					(reference "#PWR0100")
+					(reference "#PWR0101")
 					(unit 1)
 				)
@@
 		(dnp no)
 		(fields_autoplaced yes)
-		(property "Reference" "#PWR0101"
+		(property "Reference" "#PWR0102"
 			(at 39.37 139.7 0)
 			(effects
@@
 			(project "Lark"
 				(path "/a351af57-4353-47da-9f45-7393de572768/9aa817d4-eb96-4675-9e22-be0e45d55bef"
-					(reference "#PWR0101")
-					(unit 1)
-				)
+					(reference "#PWR0102")
+					(unit 1)
+				)

Commit message: started on layout, WIP
I'm not a fan of how its going, I feel like I might redo it, before I get to far into it. A patchy foundation makes an unstable house.
Connections:
- net USB_M renamed USB_N
Changed lines of the file:
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@@
 		)
 	)
-	(label "USB_M"
+	(label "USB_N"
 		(at 87.63 107.95 0)
 		(effects
@@
 		)
 	)
-	(label "USB_M"
+	(label "USB_N"
 		(at 63.5 55.88 180)
 		(effects
