File: Lark/Auxiliary.kicad_sch (KiCad schematic)
At the start: 9 parts, among them J5 0530470410, J6 0530470410, J7 0530470210

Commit message: update, WIP
- Reannotated schematic.
- Added STM32 device.
- Fixed High-side switch (removed soft-start cap for device safety).
Parts:
- renumbered D13 to D15, D14 to D16, D15 to D17, D16 to D18, J7 to J6, J5 to J7, J6 to J8, R42 to R52, R41 to R53
Connections:
- net CLK renamed SCL
Other:
- note added: "AUX 24V Power"
- note added: "Contact Rating 1 Amp Max"
- note added: "GPIO A&B Breakout"
- note added: "I2C Breakout"
- note removed: "AUX Power"
- note removed: "GPIO A&B"
- note removed: "I2C"
Changed lines of the file:
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@@
 		)
 	)
-	(text "AUX Power"
-		(exclude_from_sim no)
-		(at 260.35 17.78 0)
+	(text "AUX 24V Power"
+		(exclude_from_sim no)
+		(at 253.746 17.78 0)
 		(effects
 			(font
@@
 				(italic yes)
 			)
-		)
-	)
-	(text "GPIO A&B"
-		(exclude_from_sim no)
-		(at 24.638 85.09 0)
+			(justify left)
+		)
+	)
+	(text "GPIO A&B Breakout"
+		(exclude_from_sim no)
+		(at 19.05 85.09 0)
 		(effects
 			(font
@@
 				(italic yes)
 			)
-		)
-	)
-	(text "I2C"
-		(exclude_from_sim no)
-		(at 20.828 17.78 0)
+			(justify left)
+		)
+	)
+	(text "Contact Rating \n1 Amp Max"
+		(exclude_from_sim no)
+		(at 97.79 131.064 0)
+		(effects
+			(font
+				(size 0.762 0.762)
+			)
+		)
+	)
+	(text "Contact Rating \n1 Amp Max"
+		(exclude_from_sim no)
+		(at 273.05 54.102 0)
+		(effects
+			(font
+				(size 0.762 0.762)
+			)
+		)
+	)
+	(text "Contact Rating \n1 Amp Max"
+		(exclude_from_sim no)
+		(at 97.79 75.184 0)
+		(effects
+			(font
+				(size 0.762 0.762)
+			)
+		)
+	)
+	(text "I2C Breakout"
+		(exclude_from_sim no)
+		(at 19.05 17.78 0)
 		(effects
 			(font
@@
 				(italic yes)
 			)
+			(justify left)
 		)
 	)
@@
 		)
 	)
-	(hierarchical_label "CLK"
+	(hierarchical_label "SCL"
 		(shape input)
 		(at 30.48 49.53 180)
@@
 		(dnp no)
 		(fields_autoplaced yes)
-		(property "Reference" "#PWR0112"
+		(property "Reference" "#PWR0153"
 			(at 48.26 129.54 0)
 			(effects
@@
 			(project "Lark"
 				(path "/a351af57-4353-47da-9f45-7393de572768/f3d772fb-b064-42ef-8815-28d16dd8d37f"
-					(reference "#PWR0112")
+					(reference "#PWR0153")
 					(unit 1)
 				)
@@
 		(dnp no)
 		(fields_autoplaced yes)
-		(property "Reference" "#PWR0115"
+		(property "Reference" "#PWR0152"
 			(at 85.09 100.33 0)
 			(effects
@@
 			(project "Lark"
 				(path "/a351af57-4353-47da-9f45-7393de572768/f3d772fb-b064-42ef-8815-28d16dd8d37f"
-					(reference "#PWR0115")
+					(reference "#PWR0152")
 					(unit 1)
 				)
@@
 		(on_board yes)
 		(dnp no)
-		(property "Reference" "J6"
+		(property "Reference" "J8"
 			(at 93.726 99.06 0)
 			(effects
@@
 			(project "Lark"
 				(path "/a351af57-4353-47da-9f45-7393de572768/f3d772fb-b064-42ef-8815-28d16dd8d37f"
-					(reference "J6")
+					(reference "J8")
 					(unit 1)
 				)
@@
 		(dnp no)
 		(fields_autoplaced yes)
-		(property "Reference" "D13"
+		(property "Reference" "D15"
 			(at 50.8 56.6101 90)
 			(effects
@@
 			(project "Lark"
 				(path "/a351af57-4353-47da-9f45-7393de572768/f3d772fb-b064-42ef-8815-28d16dd8d37f"
-					(reference "D13")
+					(reference "D15")
 					(unit 1)
 				)
@@
 		(dnp no)
 		(fields_autoplaced yes)
-		(property "Reference" "D14"
+		(property "Reference" "D16"
 			(at 69.85 56.6101 90)
 			(effects
@@
 			(project "Lark"
 				(path "/a351af57-4353-47da-9f45-7393de572768/f3d772fb-b064-42ef-8815-28d16dd8d37f"
-					(reference "D14")
+					(reference "D16")
 					(unit 1)
 				)
@@
 		(dnp no)
 		(fields_autoplaced yes)
-		(property "Reference" "D16"
+		(property "Reference" "D18"
 			(at 69.85 113.7601 90)
 			(effects
@@
 			(project "Lark"
 				(path "/a351af57-4353-47da-9f45-7393de572768/f3d772fb-b064-42ef-8815-28d16dd8d37f"
-					(reference "D16")
+					(reference "D18")
 					(unit 1)
 				)
@@
 		(dnp no)
 		(fields_autoplaced yes)
-		(property "Reference" "#PWR0108"
+		(property "Reference" "#PWR0151"
 			(at 85.09 72.39 0)
 			(effects
@@
 			(project "Lark"
 				(path "/a351af57-4353-47da-9f45-7393de572768/f3d772fb-b064-42ef-8815-28d16dd8d37f"
-					(reference "#PWR0108")
+					(reference "#PWR0151")
 					(unit 1)
 				)
@@
 		(dnp no)
 		(fields_autoplaced yes)
-		(property "Reference" "#PWR0114"
+		(property "Reference" "#PWR0154"
 			(at 67.31 129.54 0)
 			(effects
@@
 			(project "Lark"
 				(path "/a351af57-4353-47da-9f45-7393de572768/f3d772fb-b064-42ef-8815-28d16dd8d37f"
-					(reference "#PWR0114")
+					(reference "#PWR0154")
 					(unit 1)
 				)
@@
 		(dnp no)
 		(fields_autoplaced yes)
-		(property "Reference" "#PWR0105"
+		(property "Reference" "#PWR0145"
 			(at 48.26 33.02 0)
 			(effects
@@
 			(project "Lark"
 				(path "/a351af57-4353-47da-9f45-7393de572768/f3d772fb-b064-42ef-8815-28d16dd8d37f"
-					(reference "#PWR0105")
+					(reference "#PWR0145")
 					(unit 1)
 				)
@@
 		(dnp no)
 		(fields_autoplaced yes)
-		(property "Reference" "D15"
+		(property "Reference" "D17"
 			(at 50.8 113.7601 90)
 			(effects
@@
 			(project "Lark"
 				(path "/a351af57-4353-47da-9f45-7393de572768/f3d772fb-b064-42ef-8815-28d16dd8d37f"
-					(reference "D15")
+					(reference "D17")
 					(unit 1)
 				)
@@
 		(on_board yes)
 		(dnp no)
-		(property "Reference" "R41"
+		(property "Reference" "R53"
 			(at 69.85 36.8299 0)
 			(effects
@@
 			(project "Lark"
 				(path "/a351af57-4353-47da-9f45-7393de572768/f3d772fb-b064-42ef-8815-28d16dd8d37f"
-					(reference "R41")
+					(reference "R53")
 					(unit 1)
 				)
@@
 		(on_board yes)
 		(dnp no)
-		(property "Reference" "J5"
+		(property "Reference" "J7"
 			(at 93.726 41.91 0)
 			(effects
@@
 			(project ""
 				(path "/a351af57-4353-47da-9f45-7393de572768/f3d772fb-b064-42ef-8815-28d16dd8d37f"
-					(reference "J5")
+					(reference "J7")
 					(unit 1)
 				)
@@
 		(on_board yes)
 		(dnp no)
-		(property "Reference" "J7"
+		(property "Reference" "J6"
 			(at 267.97 34.29 0)
 			(effects
@@
 			(project ""
 				(path "/a351af57-4353-47da-9f45-7393de572768/f3d772fb-b064-42ef-8815-28d16dd8d37f"
-					(reference "J7")
+					(reference "J6")
 					(unit 1)
 				)
@@
 		(dnp no)
 		(fields_autoplaced yes)
-		(property "Reference" "#PWR0106"
+		(property "Reference" "#PWR0146"
 			(at 67.31 33.02 0)
 			(effects
@@
 			(project "Lark"
 				(path "/a351af57-4353-47da-9f45-7393de572768/f3d772fb-b064-42ef-8815-28d16dd8d37f"
-					(reference "#PWR0106")
+					(reference "#PWR0146")
 					(unit 1)
 				)
@@
 		(dnp no)
 		(fields_autoplaced yes)
-		(property "Reference" "#PWR0107"
+		(property "Reference" "#PWR0147"
 			(at 85.09 33.02 0)
 			(effects
@@
 			(project "Lark"
 				(path "/a351af57-4353-47da-9f45-7393de572768/f3d772fb-b064-42ef-8815-28d16dd8d37f"
-					(reference "#PWR0107")
+					(reference "#PWR0147")
 					(unit 1)
 				)
@@
 		(on_board yes)
 		(dnp no)
-		(property "Reference" "R42"
+		(property "Reference" "R52"
 			(at 50.8 36.8299 0)
 			(effects
@@
 			(project "Lark"
 				(path "/a351af57-4353-47da-9f45-7393de572768/f3d772fb-b064-42ef-8815-28d16dd8d37f"
-					(reference "R42")
+					(reference "R52")
 					(unit 1)
 				)
@@
 		(dnp no)
 		(fields_autoplaced yes)
-		(property "Reference" "#PWR0110"
+		(property "Reference" "#PWR0150"
 			(at 67.31 72.39 0)
 			(effects
@@
 			(project "Lark"
 				(path "/a351af57-4353-47da-9f45-7393de572768/f3d772fb-b064-42ef-8815-28d16dd8d37f"
-					(reference "#PWR0110")
+					(reference "#PWR0150")
 					(unit 1)
 				)
@@
 		(dnp no)
 		(fields_autoplaced yes)
-		(property "Reference" "#PWR0104"
+		(property "Reference" "#PWR0144"
 			(at 259.08 31.75 0)
 			(effects
@@
 			(project "Lark"
 				(path "/a351af57-4353-47da-9f45-7393de572768/f3d772fb-b064-42ef-8815-28d16dd8d37f"
-					(reference "#PWR0104")
+					(reference "#PWR0144")
 					(unit 1)
 				)
@@
 		(dnp no)
 		(fields_autoplaced yes)
-		(property "Reference" "#PWR0109"
+		(property "Reference" "#PWR0149"
 			(at 48.26 72.39 0)
 			(effects
@@
 			(project "Lark"
 				(path "/a351af57-4353-47da-9f45-7393de572768/f3d772fb-b064-42ef-8815-28d16dd8d37f"
-					(reference "#PWR0109")
+					(reference "#PWR0149")
 					(unit 1)
 				)
@@
 		(dnp no)
 		(fields_autoplaced yes)
-		(property "Reference" "#PWR0111"
+		(property "Reference" "#PWR0148"
 			(at 259.08 53.34 0)
 			(effects
@@
 			(project "Lark"
 				(path "/a351af57-4353-47da-9f45-7393de572768/f3d772fb-b064-42ef-8815-28d16dd8d37f"
-					(reference "#PWR0111")
+					(reference "#PWR0148")
 					(unit 1)
 				)
@@
 		(dnp no)
 		(fields_autoplaced yes)
-		(property "Reference" "#PWR0116"
+		(property "Reference" "#PWR0155"
 			(at 85.09 129.54 0)
 			(effects
@@
 			(project "Lark"
 				(path "/a351af57-4353-47da-9f45-7393de572768/f3d772fb-b064-42ef-8815-28d16dd8d37f"
-					(reference "#PWR0116")
-					(unit 1)
-				)
+					(reference "#PWR0155")
+					(unit 1)
+				)

Commit message: Updated schematic, WIP
- Added NOR flash part.
- Added new CubeMX config file.
- Reannotated the schematic.
- Made some more connections to the MCU.
Parts:
- renumbered R52 to R53, R53 to R54
Changed lines of the file:
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@@
 		(on_board yes)
 		(dnp no)
-		(property "Reference" "R53"
+		(property "Reference" "R54"
 			(at 69.85 36.8299 0)
 			(effects
@@
 			(project "Lark"
 				(path "/a351af57-4353-47da-9f45-7393de572768/f3d772fb-b064-42ef-8815-28d16dd8d37f"
-					(reference "R53")
+					(reference "R54")
 					(unit 1)
 				)
@@
 		(on_board yes)
 		(dnp no)
-		(property "Reference" "R52"
+		(property "Reference" "R53"
 			(at 50.8 36.8299 0)
 			(effects
@@
 			(project "Lark"
 				(path "/a351af57-4353-47da-9f45-7393de572768/f3d772fb-b064-42ef-8815-28d16dd8d37f"
-					(reference "R52")
-					(unit 1)
-				)
+					(reference "R53")
+					(unit 1)
+				)

Commit message: Update, WIP
- Added TVS diode to 24v Supply.
- Fixed bleeder circuit at some point (I think it was this commit)
- Added Jumper to connect NTC to ADC. (again I think it was this commit)
Parts:
- renumbered D15 to D16, D16 to D17, D17 to D18, D18 to D19, R53 to R56, R54 to R57
Changed lines of the file:
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@@
 		(dnp no)
 		(fields_autoplaced yes)
-		(property "Reference" "#PWR0153"
+		(property "Reference" "#PWR0157"
 			(at 48.26 129.54 0)
 			(effects
@@
 			(project "Lark"
 				(path "/a351af57-4353-47da-9f45-7393de572768/f3d772fb-b064-42ef-8815-28d16dd8d37f"
-					(reference "#PWR0153")
+					(reference "#PWR0157")
 					(unit 1)
 				)
@@
 		(dnp no)
 		(fields_autoplaced yes)
-		(property "Reference" "#PWR0152"
+		(property "Reference" "#PWR0156"
 			(at 85.09 100.33 0)
 			(effects
@@
 			(project "Lark"
 				(path "/a351af57-4353-47da-9f45-7393de572768/f3d772fb-b064-42ef-8815-28d16dd8d37f"
-					(reference "#PWR0152")
+					(reference "#PWR0156")
 					(unit 1)
 				)
@@
 		(dnp no)
 		(fields_autoplaced yes)
-		(property "Reference" "D15"
+		(property "Reference" "D16"
 			(at 50.8 56.6101 90)
 			(effects
@@
 			(project "Lark"
 				(path "/a351af57-4353-47da-9f45-7393de572768/f3d772fb-b064-42ef-8815-28d16dd8d37f"
-					(reference "D15")
+					(reference "D16")
 					(unit 1)
 				)
@@
 		(dnp no)
 		(fields_autoplaced yes)
-		(property "Reference" "D16"
+		(property "Reference" "D17"
 			(at 69.85 56.6101 90)
 			(effects
@@
 			(project "Lark"
 				(path "/a351af57-4353-47da-9f45-7393de572768/f3d772fb-b064-42ef-8815-28d16dd8d37f"
-					(reference "D16")
+					(reference "D17")
 					(unit 1)
 				)
@@
 		(dnp no)
 		(fields_autoplaced yes)
-		(property "Reference" "D18"
+		(property "Reference" "D19"
 			(at 69.85 113.7601 90)
 			(effects
@@
 			(project "Lark"
 				(path "/a351af57-4353-47da-9f45-7393de572768/f3d772fb-b064-42ef-8815-28d16dd8d37f"
-					(reference "D18")
+					(reference "D19")
 					(unit 1)
 				)
@@
 		(dnp no)
 		(fields_autoplaced yes)
-		(property "Reference" "#PWR0151"
+		(property "Reference" "#PWR0155"
 			(at 85.09 72.39 0)
 			(effects
@@
 			(project "Lark"
 				(path "/a351af57-4353-47da-9f45-7393de572768/f3d772fb-b064-42ef-8815-28d16dd8d37f"
-					(reference "#PWR0151")
+					(reference "#PWR0155")
 					(unit 1)
 				)
@@
 		(dnp no)
 		(fields_autoplaced yes)
-		(property "Reference" "#PWR0154"
+		(property "Reference" "#PWR0158"
 			(at 67.31 129.54 0)
 			(effects
@@
 			(project "Lark"
 				(path "/a351af57-4353-47da-9f45-7393de572768/f3d772fb-b064-42ef-8815-28d16dd8d37f"
-					(reference "#PWR0154")
+					(reference "#PWR0158")
 					(unit 1)
 				)
@@
 		(dnp no)
 		(fields_autoplaced yes)
-		(property "Reference" "#PWR0145"
+		(property "Reference" "#PWR0149"
 			(at 48.26 33.02 0)
 			(effects
@@
 			(project "Lark"
 				(path "/a351af57-4353-47da-9f45-7393de572768/f3d772fb-b064-42ef-8815-28d16dd8d37f"
-					(reference "#PWR0145")
+					(reference "#PWR0149")
 					(unit 1)
 				)
@@
 		(dnp no)
 		(fields_autoplaced yes)
-		(property "Reference" "D17"
+		(property "Reference" "D18"
 			(at 50.8 113.7601 90)
 			(effects
@@
 			(project "Lark"
 				(path "/a351af57-4353-47da-9f45-7393de572768/f3d772fb-b064-42ef-8815-28d16dd8d37f"
-					(reference "D17")
+					(reference "D18")
 					(unit 1)
 				)
@@
 		(on_board yes)
 		(dnp no)
-		(property "Reference" "R54"
+		(property "Reference" "R57"
 			(at 69.85 36.8299 0)
 			(effects
@@
 			(project "Lark"
 				(path "/a351af57-4353-47da-9f45-7393de572768/f3d772fb-b064-42ef-8815-28d16dd8d37f"
-					(reference "R54")
+					(reference "R57")
 					(unit 1)
 				)
@@
 		(dnp no)
 		(fields_autoplaced yes)
-		(property "Reference" "#PWR0146"
+		(property "Reference" "#PWR0150"
 			(at 67.31 33.02 0)
 			(effects
@@
 			(project "Lark"
 				(path "/a351af57-4353-47da-9f45-7393de572768/f3d772fb-b064-42ef-8815-28d16dd8d37f"
-					(reference "#PWR0146")
+					(reference "#PWR0150")
 					(unit 1)
 				)
@@
 		(dnp no)
 		(fields_autoplaced yes)
-		(property "Reference" "#PWR0147"
+		(property "Reference" "#PWR0151"
 			(at 85.09 33.02 0)
 			(effects
@@
 			(project "Lark"
 				(path "/a351af57-4353-47da-9f45-7393de572768/f3d772fb-b064-42ef-8815-28d16dd8d37f"
-					(reference "#PWR0147")
+					(reference "#PWR0151")
 					(unit 1)
 				)
@@
 		(on_board yes)
 		(dnp no)
-		(property "Reference" "R53"
+		(property "Reference" "R56"
 			(at 50.8 36.8299 0)
 			(effects
@@
 			(project "Lark"
 				(path "/a351af57-4353-47da-9f45-7393de572768/f3d772fb-b064-42ef-8815-28d16dd8d37f"
-					(reference "R53")
+					(reference "R56")
 					(unit 1)
 				)
@@
 		(dnp no)
 		(fields_autoplaced yes)
-		(property "Reference" "#PWR0150"
+		(property "Reference" "#PWR0154"
 			(at 67.31 72.39 0)
 			(effects
@@
 			(project "Lark"
 				(path "/a351af57-4353-47da-9f45-7393de572768/f3d772fb-b064-42ef-8815-28d16dd8d37f"
-					(reference "#PWR0150")
+					(reference "#PWR0154")
 					(unit 1)
 				)
@@
 		(dnp no)
 		(fields_autoplaced yes)
-		(property "Reference" "#PWR0144"
+		(property "Reference" "#PWR0148"
 			(at 259.08 31.75 0)
 			(effects
@@
 			(project "Lark"
 				(path "/a351af57-4353-47da-9f45-7393de572768/f3d772fb-b064-42ef-8815-28d16dd8d37f"
-					(reference "#PWR0144")
+					(reference "#PWR0148")
 					(unit 1)
 				)
@@
 		(dnp no)
 		(fields_autoplaced yes)
-		(property "Reference" "#PWR0149"
+		(property "Reference" "#PWR0153"
 			(at 48.26 72.39 0)
 			(effects
@@
 			(project "Lark"
 				(path "/a351af57-4353-47da-9f45-7393de572768/f3d772fb-b064-42ef-8815-28d16dd8d37f"
-					(reference "#PWR0149")
+					(reference "#PWR0153")
 					(unit 1)
 				)
@@
 		(dnp no)
 		(fields_autoplaced yes)
-		(property "Reference" "#PWR0148"
+		(property "Reference" "#PWR0152"
 			(at 259.08 53.34 0)
 			(effects
@@
 			(project "Lark"
 				(path "/a351af57-4353-47da-9f45-7393de572768/f3d772fb-b064-42ef-8815-28d16dd8d37f"
-					(reference "#PWR0148")
+					(reference "#PWR0152")
 					(unit 1)
 				)
@@
 		(dnp no)
 		(fields_autoplaced yes)
-		(property "Reference" "#PWR0155"
+		(property "Reference" "#PWR0159"
 			(at 85.09 129.54 0)
 			(effects
@@
 			(project "Lark"
 				(path "/a351af57-4353-47da-9f45-7393de572768/f3d772fb-b064-42ef-8815-28d16dd8d37f"
-					(reference "#PWR0155")
-					(unit 1)
-				)
+					(reference "#PWR0159")
+					(unit 1)
+				)

Commit message: updated WIP
- fixed high-side switch (swapped out pfets)
- swapped out bleeder fet.
- changed a few footprints.
- changed zeners to 15v ones
- added soft-start cap back in to the high-side switch.

(today ive mainly been struggling with the inrush current, but I think its solved now)
Parts:
- renumbered D16 to D18, D17 to D19, D18 to D20, D19 to D21
Changed lines of the file:
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@@
 		(dnp no)
 		(fields_autoplaced yes)
-		(property "Reference" "#PWR0157"
+		(property "Reference" "#PWR0158"
 			(at 48.26 129.54 0)
 			(effects
@@
 			(project "Lark"
 				(path "/a351af57-4353-47da-9f45-7393de572768/f3d772fb-b064-42ef-8815-28d16dd8d37f"
-					(reference "#PWR0157")
+					(reference "#PWR0158")
 					(unit 1)
 				)
@@
 		(dnp no)
 		(fields_autoplaced yes)
-		(property "Reference" "#PWR0156"
+		(property "Reference" "#PWR0157"
 			(at 85.09 100.33 0)
 			(effects
@@
 			(project "Lark"
 				(path "/a351af57-4353-47da-9f45-7393de572768/f3d772fb-b064-42ef-8815-28d16dd8d37f"
-					(reference "#PWR0156")
+					(reference "#PWR0157")
 					(unit 1)
 				)
@@
 		(dnp no)
 		(fields_autoplaced yes)
-		(property "Reference" "D16"
+		(property "Reference" "D18"
 			(at 50.8 56.6101 90)
 			(effects
@@
 			(project "Lark"
 				(path "/a351af57-4353-47da-9f45-7393de572768/f3d772fb-b064-42ef-8815-28d16dd8d37f"
-					(reference "D16")
+					(reference "D18")
 					(unit 1)
 				)
@@
 		(dnp no)
 		(fields_autoplaced yes)
-		(property "Reference" "D17"
+		(property "Reference" "D19"
 			(at 69.85 56.6101 90)
 			(effects
@@
 			(project "Lark"
 				(path "/a351af57-4353-47da-9f45-7393de572768/f3d772fb-b064-42ef-8815-28d16dd8d37f"
-					(reference "D17")
+					(reference "D19")
 					(unit 1)
 				)
@@
 		(dnp no)
 		(fields_autoplaced yes)
-		(property "Reference" "D19"
+		(property "Reference" "D21"
 			(at 69.85 113.7601 90)
 			(effects
@@
 			(project "Lark"
 				(path "/a351af57-4353-47da-9f45-7393de572768/f3d772fb-b064-42ef-8815-28d16dd8d37f"
-					(reference "D19")
+					(reference "D21")
 					(unit 1)
 				)
@@
 		(dnp no)
 		(fields_autoplaced yes)
-		(property "Reference" "#PWR0155"
+		(property "Reference" "#PWR0156"
 			(at 85.09 72.39 0)
 			(effects
@@
 			(project "Lark"
 				(path "/a351af57-4353-47da-9f45-7393de572768/f3d772fb-b064-42ef-8815-28d16dd8d37f"
-					(reference "#PWR0155")
+					(reference "#PWR0156")
 					(unit 1)
 				)
@@
 		(dnp no)
 		(fields_autoplaced yes)
-		(property "Reference" "#PWR0158"
+		(property "Reference" "#PWR0159"
 			(at 67.31 129.54 0)
 			(effects
@@
 			(project "Lark"
 				(path "/a351af57-4353-47da-9f45-7393de572768/f3d772fb-b064-42ef-8815-28d16dd8d37f"
-					(reference "#PWR0158")
+					(reference "#PWR0159")
 					(unit 1)
 				)
@@
 		(dnp no)
 		(fields_autoplaced yes)
-		(property "Reference" "#PWR0149"
+		(property "Reference" "#PWR0150"
 			(at 48.26 33.02 0)
 			(effects
@@
 			(project "Lark"
 				(path "/a351af57-4353-47da-9f45-7393de572768/f3d772fb-b064-42ef-8815-28d16dd8d37f"
-					(reference "#PWR0149")
+					(reference "#PWR0150")
 					(unit 1)
 				)
@@
 		(dnp no)
 		(fields_autoplaced yes)
-		(property "Reference" "D18"
+		(property "Reference" "D20"
 			(at 50.8 113.7601 90)
 			(effects
@@
 			(project "Lark"
 				(path "/a351af57-4353-47da-9f45-7393de572768/f3d772fb-b064-42ef-8815-28d16dd8d37f"
-					(reference "D18")
+					(reference "D20")
 					(unit 1)
 				)
@@
 		(dnp no)
 		(fields_autoplaced yes)
-		(property "Reference" "#PWR0150"
+		(property "Reference" "#PWR0151"
 			(at 67.31 33.02 0)
 			(effects
@@
 			(project "Lark"
 				(path "/a351af57-4353-47da-9f45-7393de572768/f3d772fb-b064-42ef-8815-28d16dd8d37f"
-					(reference "#PWR0150")
+					(reference "#PWR0151")
 					(unit 1)
 				)
@@
 		(dnp no)
 		(fields_autoplaced yes)
-		(property "Reference" "#PWR0151"
+		(property "Reference" "#PWR0152"
 			(at 85.09 33.02 0)
 			(effects
@@
 			(project "Lark"
 				(path "/a351af57-4353-47da-9f45-7393de572768/f3d772fb-b064-42ef-8815-28d16dd8d37f"
-					(reference "#PWR0151")
+					(reference "#PWR0152")
 					(unit 1)
 				)
@@
 		(dnp no)
 		(fields_autoplaced yes)
-		(property "Reference" "#PWR0154"
+		(property "Reference" "#PWR0155"
 			(at 67.31 72.39 0)
 			(effects
@@
 			(project "Lark"
 				(path "/a351af57-4353-47da-9f45-7393de572768/f3d772fb-b064-42ef-8815-28d16dd8d37f"
-					(reference "#PWR0154")
+					(reference "#PWR0155")
 					(unit 1)
 				)
@@
 		(dnp no)
 		(fields_autoplaced yes)
-		(property "Reference" "#PWR0148"
+		(property "Reference" "#PWR0149"
 			(at 259.08 31.75 0)
 			(effects
@@
 			(project "Lark"
 				(path "/a351af57-4353-47da-9f45-7393de572768/f3d772fb-b064-42ef-8815-28d16dd8d37f"
-					(reference "#PWR0148")
+					(reference "#PWR0149")
 					(unit 1)
 				)
@@
 		(dnp no)
 		(fields_autoplaced yes)
-		(property "Reference" "#PWR0153"
+		(property "Reference" "#PWR0154"
 			(at 48.26 72.39 0)
 			(effects
@@
 			(project "Lark"
 				(path "/a351af57-4353-47da-9f45-7393de572768/f3d772fb-b064-42ef-8815-28d16dd8d37f"
-					(reference "#PWR0153")
+					(reference "#PWR0154")
 					(unit 1)
 				)
@@
 		(dnp no)
 		(fields_autoplaced yes)
-		(property "Reference" "#PWR0152"
+		(property "Reference" "#PWR0153"
 			(at 259.08 53.34 0)
 			(effects
@@
 			(project "Lark"
 				(path "/a351af57-4353-47da-9f45-7393de572768/f3d772fb-b064-42ef-8815-28d16dd8d37f"
-					(reference "#PWR0152")
+					(reference "#PWR0153")
 					(unit 1)
 				)
@@
 		(dnp no)
 		(fields_autoplaced yes)
-		(property "Reference" "#PWR0159"
+		(property "Reference" "#PWR0160"
 			(at 85.09 129.54 0)
 			(effects
@@
 			(project "Lark"
 				(path "/a351af57-4353-47da-9f45-7393de572768/f3d772fb-b064-42ef-8815-28d16dd8d37f"
-					(reference "#PWR0159")
-					(unit 1)
-				)
+					(reference "#PWR0160")
+					(unit 1)
+				)
