File: Lark/Boot_Controller.kicad_sch (KiCad schematic)
At the start: 12 parts, among them J2 0530470210, SW1 PTS636 SP50 SMTR LFS, U7 ATTINY85-20PU, U8 ATTINY85-20SU

Commit message: added power section to schematic
It needs revised, due to thermal issue. Specifically in regards to my soft start circuit, the mosfet wont be able to handle the power dissipated during a slow turn on.
Parts:
- C12, C13: value 0.1 µF -> 0.1µF
- D5: footprint onsemi:D_SOD-523 -> onsemi:ESD5Z3.3T1G
Changed lines of the file:
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@@
 			)
 		)
-		(property "Value" "0.1 µF"
+		(property "Value" "0.1µF"
 			(at 267.97 110.4962 0)
 			(effects
@@
 			)
 		)
-		(property "Datasheet" "https://search.murata.co.jp/Ceramy/image/img/A01X/G101/ENG/GRM188R72A104MA35-01A.pdf"
+		(property "Datasheet" "~"
 			(at 265.43 109.22 0)
 			(effects
@@
 			)
 		)
-		(property "Footprint" "onsemi:D_SOD-523"
+		(property "Footprint" "onsemi:ESD5Z3.3T1G"
 			(at 45.72 172.72 0)
 			(effects
@@
 			)
 		)
-		(property "Datasheet" "https://www.seielect.com/catalog/SEI-RMCF_RMCP.pdf"
+		(property "Datasheet" "~"
 			(at 26.67 95.25 0)
 			(effects
@@
 			)
 		)
-		(property "Value" "0.1 µF"
+		(property "Value" "0.1µF"
 			(at 68.58 172.7262 0)
 			(effects
@@
 			)
 		)
-		(property "Datasheet" "https://search.murata.co.jp/Ceramy/image/img/A01X/G101/ENG/GRM188R72A104MA35-01A.pdf"
+		(property "Datasheet" "~"
 			(at 66.04 171.45 0)
 			(effects
@@
 			)
 		)
-		(property "Datasheet" "https://www.seielect.com/catalog/SEI-RMCF_RMCP.pdf"
+		(property "Datasheet" "~"
 			(at 55.88 163.83 0)
 			(effects
@@
 			)
 		)
-		(property "Description" "Generic connector, single row, 01x02, script generated"
+		(property "Description" "Connector Header Through Hole 2 position 0.049\" (1.25mm)"
 			(at 26.67 171.45 0)
 			(effects
@@
 			)
 		)
-		(property "Datasheet" "https://www.seielect.com/catalog/SEI-RMCF_RMCP.pdf"
+		(property "Datasheet" "~"
 			(at 66.04 154.94 0)
 			(effects
@@
 			)
 		)
-		(property "Datasheet" "https://www.seielect.com/catalog/SEI-RMCF_RMCP.pdf"
+		(property "Datasheet" "~"
 			(at 36.83 107.95 0)
 			(effects

Commit message: update, WIP
- Reannotated schematic.
- Added STM32 device.
- Fixed High-side switch (removed soft-start cap for device safety).
Parts:
- renumbered C12 to C24, C13 to C25, D6 to D7, D5 to D8, J2 to J3, R26 to R37, R29 to R38, R27 to R39, R28 to R40, U8 to U10, U7 to U11
Changed lines of the file:
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@@
 		(dnp no)
 		(fields_autoplaced yes)
-		(property "Reference" "#PWR067"
+		(property "Reference" "#PWR098"
 			(at 265.43 35.56 0)
 			(effects
@@
 			(project "Lark"
 				(path "/a351af57-4353-47da-9f45-7393de572768/edc369e3-0a21-4448-a6d2-131219450aa0"
-					(reference "#PWR067")
+					(reference "#PWR098")
 					(unit 1)
 				)
@@
 		(on_board yes)
 		(dnp no)
-		(property "Reference" "C12"
+		(property "Reference" "C24"
 			(at 267.97 107.9562 0)
 			(effects
@@
 			(project "Lark"
 				(path "/a351af57-4353-47da-9f45-7393de572768/edc369e3-0a21-4448-a6d2-131219450aa0"
-					(reference "C12")
+					(reference "C24")
 					(unit 1)
 				)
@@
 		(dnp no)
 		(fields_autoplaced yes)
-		(property "Reference" "#PWR059"
+		(property "Reference" "#PWR0103"
 			(at 265.43 130.81 0)
 			(effects
@@
 			(project "Lark"
 				(path "/a351af57-4353-47da-9f45-7393de572768/edc369e3-0a21-4448-a6d2-131219450aa0"
-					(reference "#PWR059")
+					(reference "#PWR0103")
 					(unit 1)
 				)
@@
 		(dnp no)
 		(fields_autoplaced yes)
-		(property "Reference" "#PWR068"
+		(property "Reference" "#PWR099"
 			(at 265.43 66.04 0)
 			(effects
@@
 			(project "Lark"
 				(path "/a351af57-4353-47da-9f45-7393de572768/edc369e3-0a21-4448-a6d2-131219450aa0"
-					(reference "#PWR068")
+					(reference "#PWR099")
 					(unit 1)
 				)
@@
 		(on_board yes)
 		(dnp no)
-		(property "Reference" "U8"
+		(property "Reference" "U10"
 			(at 246.126 34.29 0)
 			(effects
@@
 			(project "Lark"
 				(path "/a351af57-4353-47da-9f45-7393de572768/edc369e3-0a21-4448-a6d2-131219450aa0"
-					(reference "U8")
+					(reference "U10")
 					(unit 1)
 				)
@@
 		(dnp no)
 		(fields_autoplaced yes)
-		(property "Reference" "#PWR065"
+		(property "Reference" "#PWR0106"
 			(at 38.1 186.69 0)
 			(effects
@@
 			(project "Lark"
 				(path "/a351af57-4353-47da-9f45-7393de572768/edc369e3-0a21-4448-a6d2-131219450aa0"
-					(reference "#PWR065")
+					(reference "#PWR0106")
 					(unit 1)
 				)
@@
 		(dnp no)
 		(fields_autoplaced yes)
-		(property "Reference" "D5"
+		(property "Reference" "D8"
 			(at 48.26 172.1801 90)
 			(effects
@@
 			(project "Lark"
 				(path "/a351af57-4353-47da-9f45-7393de572768/edc369e3-0a21-4448-a6d2-131219450aa0"
-					(reference "D5")
+					(reference "D8")
 					(unit 1)
 				)
@@
 		(on_board yes)
 		(dnp no)
-		(property "Reference" "R26"
+		(property "Reference" "R37"
 			(at 29.21 93.9799 0)
 			(effects
@@
 			(project "Lark"
 				(path "/a351af57-4353-47da-9f45-7393de572768/edc369e3-0a21-4448-a6d2-131219450aa0"
-					(reference "R26")
+					(reference "R37")
 					(unit 1)
 				)
@@
 		(on_board yes)
 		(dnp no)
-		(property "Reference" "C13"
+		(property "Reference" "C25"
 			(at 68.58 170.1862 0)
 			(effects
@@
 			(project "Lark"
 				(path "/a351af57-4353-47da-9f45-7393de572768/edc369e3-0a21-4448-a6d2-131219450aa0"
-					(reference "C13")
+					(reference "C25")
 					(unit 1)
 				)
@@
 		(dnp no)
 		(fields_autoplaced yes)
-		(property "Reference" "#PWR063"
+		(property "Reference" "#PWR0107"
 			(at 45.72 186.69 0)
 			(effects
@@
 			(project "Lark"
 				(path "/a351af57-4353-47da-9f45-7393de572768/edc369e3-0a21-4448-a6d2-131219450aa0"
-					(reference "#PWR063")
+					(reference "#PWR0107")
 					(unit 1)
 				)
@@
 		(on_board yes)
 		(dnp no)
-		(property "Reference" "R28"
+		(property "Reference" "R40"
 			(at 56.896 161.29 90)
 			(effects
@@
 			(project "Lark"
 				(path "/a351af57-4353-47da-9f45-7393de572768/edc369e3-0a21-4448-a6d2-131219450aa0"
-					(reference "R28")
+					(reference "R40")
 					(unit 1)
 				)
@@
 		(dnp no)
 		(fields_autoplaced yes)
-		(property "Reference" "#PWR060"
+		(property "Reference" "#PWR0100"
 			(at 26.67 90.17 0)
 			(effects
@@
 			(project "Lark"
 				(path "/a351af57-4353-47da-9f45-7393de572768/edc369e3-0a21-4448-a6d2-131219450aa0"
-					(reference "#PWR060")
+					(reference "#PWR0100")
 					(unit 1)
 				)
@@
 		(dnp no)
 		(fields_autoplaced yes)
-		(property "Reference" "#PWR061"
+		(property "Reference" "#PWR0104"
 			(at 66.04 151.13 0)
 			(effects
@@
 			(project "Lark"
 				(path "/a351af57-4353-47da-9f45-7393de572768/edc369e3-0a21-4448-a6d2-131219450aa0"
-					(reference "#PWR061")
+					(reference "#PWR0104")
 					(unit 1)
 				)
@@
 		(dnp no)
 		(fields_autoplaced yes)
-		(property "Reference" "#PWR064"
+		(property "Reference" "#PWR0101"
 			(at 36.83 90.17 0)
 			(effects
@@
 			(project "Lark"
 				(path "/a351af57-4353-47da-9f45-7393de572768/edc369e3-0a21-4448-a6d2-131219450aa0"
-					(reference "#PWR064")
+					(reference "#PWR0101")
 					(unit 1)
 				)
@@
 		(on_board yes)
 		(dnp no)
-		(property "Reference" "J2"
+		(property "Reference" "J3"
 			(at 26.162 161.29 0)
 			(effects
@@
 			(project "Lark"
 				(path "/a351af57-4353-47da-9f45-7393de572768/edc369e3-0a21-4448-a6d2-131219450aa0"
-					(reference "J2")
+					(reference "J3")
 					(unit 1)
 				)
@@
 		(on_board yes)
 		(dnp no)
-		(property "Reference" "R27"
+		(property "Reference" "R39"
 			(at 68.58 153.6699 0)
 			(effects
@@
 			(project "Lark"
 				(path "/a351af57-4353-47da-9f45-7393de572768/edc369e3-0a21-4448-a6d2-131219450aa0"
-					(reference "R27")
+					(reference "R39")
 					(unit 1)
 				)
@@
 		(dnp no)
 		(fields_autoplaced yes)
-		(property "Reference" "#PWR062"
+		(property "Reference" "#PWR0108"
 			(at 66.04 186.69 0)
 			(effects
@@
 			(project "Lark"
 				(path "/a351af57-4353-47da-9f45-7393de572768/edc369e3-0a21-4448-a6d2-131219450aa0"
-					(reference "#PWR062")
+					(reference "#PWR0108")
 					(unit 1)
 				)
@@
 		(on_board yes)
 		(dnp no)
-		(property "Reference" "R29"
+		(property "Reference" "R38"
 			(at 39.37 106.6799 0)
 			(effects
@@
 			(project "Lark"
 				(path "/a351af57-4353-47da-9f45-7393de572768/edc369e3-0a21-4448-a6d2-131219450aa0"
-					(reference "R29")
+					(reference "R38")
 					(unit 1)
 				)
@@
 		(dnp no)
 		(fields_autoplaced yes)
-		(property "Reference" "D6"
+		(property "Reference" "D7"
 			(at 40.64 95.5674 90)
 			(effects
@@
 			(project "Lark"
 				(path "/a351af57-4353-47da-9f45-7393de572768/edc369e3-0a21-4448-a6d2-131219450aa0"
-					(reference "D6")
+					(reference "D7")
 					(unit 1)
 				)
@@
 		(dnp no)
 		(fields_autoplaced yes)
-		(property "Reference" "#PWR066"
+		(property "Reference" "#PWR0105"
 			(at 26.67 156.21 0)
 			(effects
@@
 			(project "Lark"
 				(path "/a351af57-4353-47da-9f45-7393de572768/edc369e3-0a21-4448-a6d2-131219450aa0"
-					(reference "#PWR066")
+					(reference "#PWR0105")
 					(unit 1)
 				)
@@
 		(on_board yes)
 		(dnp no)
-		(property "Reference" "U7"
+		(property "Reference" "U11"
 			(at 246.38 97.79 0)
 			(effects
@@
 			(project "Lark"
 				(path "/a351af57-4353-47da-9f45-7393de572768/edc369e3-0a21-4448-a6d2-131219450aa0"
-					(reference "U7")
+					(reference "U11")
 					(unit 1)
 				)
@@
 		(dnp no)
 		(fields_autoplaced yes)
-		(property "Reference" "#PWR058"
+		(property "Reference" "#PWR0102"
 			(at 265.43 100.33 0)
 			(effects
@@
 			(project "Lark"
 				(path "/a351af57-4353-47da-9f45-7393de572768/edc369e3-0a21-4448-a6d2-131219450aa0"
-					(reference "#PWR058")
-					(unit 1)
-				)
+					(reference "#PWR0102")
+					(unit 1)
+				)

Commit message: Updated schematic, WIP
- Added NOR flash part.
- Added new CubeMX config file.
- Reannotated the schematic.
- Made some more connections to the MCU.
Parts:
- U10: now not fitted
- renumbered R37 to R38, R38 to R39, R39 to R40, R40 to R41
Other:
- moved on the sheet: C24, U11

Commit message: Update, WIP
- Added TVS diode to 24v Supply.
- Fixed bleeder circuit at some point (I think it was this commit)
- Added Jumper to connect NTC to ADC. (again I think it was this commit)
Parts:
- renumbered D7 to D8, D8 to D9, R38 to R41, R39 to R42, R40 to R43, R41 to R44
Changed lines of the file:
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@@
 	(wire
 		(pts
-			(xy 26.67 119.38) (xy 53.34 119.38)
+			(xy 26.67 119.38) (xy 59.69 119.38)
 		)
 		(stroke
@@
 	(wire
 		(pts
-			(xy 36.83 115.57) (xy 53.34 115.57)
+			(xy 36.83 115.57) (xy 59.69 115.57)
 		)
 		(stroke
@@
 	)
 	(label "IO3"
-		(at 53.34 115.57 180)
+		(at 59.69 115.57 180)
 		(effects
 			(font
@@
 	)
 	(label "MCURST"
-		(at 53.34 119.38 180)
+		(at 59.69 119.38 180)
 		(effects
 			(font
@@
 		(dnp no)
 		(fields_autoplaced yes)
-		(property "Reference" "#PWR098"
+		(property "Reference" "#PWR0102"
 			(at 266.7 34.29 0)
 			(effects
@@
 			(project "Lark"
 				(path "/a351af57-4353-47da-9f45-7393de572768/edc369e3-0a21-4448-a6d2-131219450aa0"
-					(reference "#PWR098")
+					(reference "#PWR0102")
 					(unit 1)
 				)
@@
 		(dnp no)
 		(fields_autoplaced yes)
-		(property "Reference" "#PWR0105"
+		(property "Reference" "#PWR0109"
 			(at 266.7 156.21 0)
 			(effects
@@
 			(project "Lark"
 				(path "/a351af57-4353-47da-9f45-7393de572768/edc369e3-0a21-4448-a6d2-131219450aa0"
-					(reference "#PWR0105")
+					(reference "#PWR0109")
 					(unit 1)
 				)
@@
 		(dnp no)
 		(fields_autoplaced yes)
-		(property "Reference" "#PWR099"
+		(property "Reference" "#PWR0103"
 			(at 266.7 64.77 0)
 			(effects
@@
 			(project "Lark"
 				(path "/a351af57-4353-47da-9f45-7393de572768/edc369e3-0a21-4448-a6d2-131219450aa0"
-					(reference "#PWR099")
+					(reference "#PWR0103")
 					(unit 1)
 				)
@@
 		(dnp no)
 		(fields_autoplaced yes)
-		(property "Reference" "#PWR0106"
+		(property "Reference" "#PWR0110"
 			(at 38.1 186.69 0)
 			(effects
@@
 			(project "Lark"
 				(path "/a351af57-4353-47da-9f45-7393de572768/edc369e3-0a21-4448-a6d2-131219450aa0"
-					(reference "#PWR0106")
+					(reference "#PWR0110")
 					(unit 1)
 				)
@@
 		(dnp no)
 		(fields_autoplaced yes)
-		(property "Reference" "D8"
+		(property "Reference" "D9"
 			(at 48.26 172.1801 90)
 			(effects
@@
 			(project "Lark"
 				(path "/a351af57-4353-47da-9f45-7393de572768/edc369e3-0a21-4448-a6d2-131219450aa0"
-					(reference "D8")
+					(reference "D9")
 					(unit 1)
 				)
@@
 		(on_board yes)
 		(dnp no)
-		(property "Reference" "R38"
+		(property "Reference" "R41"
 			(at 29.21 93.9799 0)
 			(effects
@@
 			(project "Lark"
 				(path "/a351af57-4353-47da-9f45-7393de572768/edc369e3-0a21-4448-a6d2-131219450aa0"
-					(reference "R38")
+					(reference "R41")
 					(unit 1)
 				)
@@
 		(dnp no)
 		(fields_autoplaced yes)
-		(property "Reference" "#PWR0107"
+		(property "Reference" "#PWR0111"
 			(at 45.72 186.69 0)
 			(effects
@@
 			(project "Lark"
 				(path "/a351af57-4353-47da-9f45-7393de572768/edc369e3-0a21-4448-a6d2-131219450aa0"
-					(reference "#PWR0107")
+					(reference "#PWR0111")
 					(unit 1)
 				)
@@
 		(on_board yes)
 		(dnp no)
-		(property "Reference" "R41"
+		(property "Reference" "R44"
 			(at 56.896 161.29 90)
 			(effects
@@
 			(project "Lark"
 				(path "/a351af57-4353-47da-9f45-7393de572768/edc369e3-0a21-4448-a6d2-131219450aa0"
-					(reference "R41")
+					(reference "R44")
 					(unit 1)
 				)
@@
 		(dnp no)
 		(fields_autoplaced yes)
-		(property "Reference" "#PWR0100"
+		(property "Reference" "#PWR0104"
 			(at 26.67 90.17 0)
 			(effects
@@
 			(project "Lark"
 				(path "/a351af57-4353-47da-9f45-7393de572768/edc369e3-0a21-4448-a6d2-131219450aa0"
-					(reference "#PWR0100")
+					(reference "#PWR0104")
 					(unit 1)
 				)
@@
 		(dnp no)
 		(fields_autoplaced yes)
-		(property "Reference" "#PWR0103"
+		(property "Reference" "#PWR0107"
 			(at 66.04 151.13 0)
 			(effects
@@
 			(project "Lark"
 				(path "/a351af57-4353-47da-9f45-7393de572768/edc369e3-0a21-4448-a6d2-131219450aa0"
-					(reference "#PWR0103")
+					(reference "#PWR0107")
 					(unit 1)
 				)
@@
 		(dnp no)
 		(fields_autoplaced yes)
-		(property "Reference" "#PWR0101"
+		(property "Reference" "#PWR0105"
 			(at 36.83 90.17 0)
 			(effects
@@
 			(project "Lark"
 				(path "/a351af57-4353-47da-9f45-7393de572768/edc369e3-0a21-4448-a6d2-131219450aa0"
-					(reference "#PWR0101")
+					(reference "#PWR0105")
 					(unit 1)
 				)
@@
 		(on_board yes)
 		(dnp no)
-		(property "Reference" "R40"
+		(property "Reference" "R43"
 			(at 68.58 153.6699 0)
 			(effects
@@
 			(project "Lark"
 				(path "/a351af57-4353-47da-9f45-7393de572768/edc369e3-0a21-4448-a6d2-131219450aa0"
-					(reference "R40")
+					(reference "R43")
 					(unit 1)
 				)
@@
 		(dnp no)
 		(fields_autoplaced yes)
-		(property "Reference" "#PWR0108"
+		(property "Reference" "#PWR0112"
 			(at 66.04 186.69 0)
 			(effects
@@
 			(project "Lark"
 				(path "/a351af57-4353-47da-9f45-7393de572768/edc369e3-0a21-4448-a6d2-131219450aa0"
-					(reference "#PWR0108")
+					(reference "#PWR0112")
 					(unit 1)
 				)
@@
 		(on_board yes)
 		(dnp no)
-		(property "Reference" "R39"
+		(property "Reference" "R42"
 			(at 39.37 106.6799 0)
 			(effects
@@
 			(project "Lark"
 				(path "/a351af57-4353-47da-9f45-7393de572768/edc369e3-0a21-4448-a6d2-131219450aa0"
-					(reference "R39")
+					(reference "R42")
 					(unit 1)
 				)
@@
 		(dnp no)
 		(fields_autoplaced yes)
-		(property "Reference" "D7"
+		(property "Reference" "D8"
 			(at 40.64 95.5674 90)
 			(effects
@@
 			(project "Lark"
 				(path "/a351af57-4353-47da-9f45-7393de572768/edc369e3-0a21-4448-a6d2-131219450aa0"
-					(reference "D7")
+					(reference "D8")
 					(unit 1)
 				)
@@
 		(dnp no)
 		(fields_autoplaced yes)
-		(property "Reference" "#PWR0104"
+		(property "Reference" "#PWR0108"
 			(at 26.67 156.21 0)
 			(effects
@@
 			(project "Lark"
 				(path "/a351af57-4353-47da-9f45-7393de572768/edc369e3-0a21-4448-a6d2-131219450aa0"
-					(reference "#PWR0104")
+					(reference "#PWR0108")
 					(unit 1)
 				)
@@
 		(dnp no)
 		(fields_autoplaced yes)
-		(property "Reference" "#PWR0102"
+		(property "Reference" "#PWR0106"
 			(at 266.7 125.73 0)
 			(effects
@@
 			(project "Lark"
 				(path "/a351af57-4353-47da-9f45-7393de572768/edc369e3-0a21-4448-a6d2-131219450aa0"
-					(reference "#PWR0102")
+					(reference "#PWR0106")
 					(unit 1)
 				)

Commit message: updated WIP
- fixed high-side switch (swapped out pfets)
- swapped out bleeder fet.
- changed a few footprints.
- changed zeners to 15v ones
- added soft-start cap back in to the high-side switch.

(today ive mainly been struggling with the inrush current, but I think its solved now)
Parts:
- renumbered C24 to C25, C25 to C26, D8 to D10, D9 to D11, U10 to U12, U11 to U13
Changed lines of the file:
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@@
 		(dnp no)
 		(fields_autoplaced yes)
-		(property "Reference" "#PWR0102"
+		(property "Reference" "#PWR0103"
 			(at 266.7 34.29 0)
 			(effects
@@
 			(project "Lark"
 				(path "/a351af57-4353-47da-9f45-7393de572768/edc369e3-0a21-4448-a6d2-131219450aa0"
-					(reference "#PWR0102")
+					(reference "#PWR0103")
 					(unit 1)
 				)
@@
 		(on_board yes)
 		(dnp no)
-		(property "Reference" "C24"
+		(property "Reference" "C25"
 			(at 269.24 133.3562 0)
 			(effects
@@
 			(project "Lark"
 				(path "/a351af57-4353-47da-9f45-7393de572768/edc369e3-0a21-4448-a6d2-131219450aa0"
-					(reference "C24")
+					(reference "C25")
 					(unit 1)
 				)
@@
 		(dnp no)
 		(fields_autoplaced yes)
-		(property "Reference" "#PWR0109"
+		(property "Reference" "#PWR0110"
 			(at 266.7 156.21 0)
 			(effects
@@
 			(project "Lark"
 				(path "/a351af57-4353-47da-9f45-7393de572768/edc369e3-0a21-4448-a6d2-131219450aa0"
-					(reference "#PWR0109")
+					(reference "#PWR0110")
 					(unit 1)
 				)
@@
 		(dnp no)
 		(fields_autoplaced yes)
-		(property "Reference" "#PWR0103"
+		(property "Reference" "#PWR0104"
 			(at 266.7 64.77 0)
 			(effects
@@
 			(project "Lark"
 				(path "/a351af57-4353-47da-9f45-7393de572768/edc369e3-0a21-4448-a6d2-131219450aa0"
-					(reference "#PWR0103")
+					(reference "#PWR0104")
 					(unit 1)
 				)
@@
 		(on_board yes)
 		(dnp yes)
-		(property "Reference" "U10"
+		(property "Reference" "U12"
 			(at 247.396 33.02 0)
 			(effects
@@
 			(project "Lark"
 				(path "/a351af57-4353-47da-9f45-7393de572768/edc369e3-0a21-4448-a6d2-131219450aa0"
-					(reference "U10")
+					(reference "U12")
 					(unit 1)
 				)
@@
 		(dnp no)
 		(fields_autoplaced yes)
-		(property "Reference" "#PWR0110"
+		(property "Reference" "#PWR0111"
 			(at 38.1 186.69 0)
 			(effects
@@
 			(project "Lark"
 				(path "/a351af57-4353-47da-9f45-7393de572768/edc369e3-0a21-4448-a6d2-131219450aa0"
-					(reference "#PWR0110")
+					(reference "#PWR0111")
 					(unit 1)
 				)
@@
 		(dnp no)
 		(fields_autoplaced yes)
-		(property "Reference" "D9"
+		(property "Reference" "D11"
 			(at 48.26 172.1801 90)
 			(effects
@@
 			(project "Lark"
 				(path "/a351af57-4353-47da-9f45-7393de572768/edc369e3-0a21-4448-a6d2-131219450aa0"
-					(reference "D9")
+					(reference "D11")
 					(unit 1)
 				)
@@
 		(on_board yes)
 		(dnp no)
-		(property "Reference" "C25"
+		(property "Reference" "C26"
 			(at 68.58 170.1862 0)
 			(effects
@@
 			(project "Lark"
 				(path "/a351af57-4353-47da-9f45-7393de572768/edc369e3-0a21-4448-a6d2-131219450aa0"
-					(reference "C25")
+					(reference "C26")
 					(unit 1)
 				)
@@
 		(dnp no)
 		(fields_autoplaced yes)
-		(property "Reference" "#PWR0111"
+		(property "Reference" "#PWR0112"
 			(at 45.72 186.69 0)
 			(effects
@@
 			(project "Lark"
 				(path "/a351af57-4353-47da-9f45-7393de572768/edc369e3-0a21-4448-a6d2-131219450aa0"
-					(reference "#PWR0111")
+					(reference "#PWR0112")
 					(unit 1)
 				)
@@
 		(dnp no)
 		(fields_autoplaced yes)
-		(property "Reference" "#PWR0104"
+		(property "Reference" "#PWR0105"
 			(at 26.67 90.17 0)
 			(effects
@@
 			(project "Lark"
 				(path "/a351af57-4353-47da-9f45-7393de572768/edc369e3-0a21-4448-a6d2-131219450aa0"
-					(reference "#PWR0104")
+					(reference "#PWR0105")
 					(unit 1)
 				)
@@
 		(dnp no)
 		(fields_autoplaced yes)
-		(property "Reference" "#PWR0107"
+		(property "Reference" "#PWR0108"
 			(at 66.04 151.13 0)
 			(effects
@@
 			(project "Lark"
 				(path "/a351af57-4353-47da-9f45-7393de572768/edc369e3-0a21-4448-a6d2-131219450aa0"
-					(reference "#PWR0107")
+					(reference "#PWR0108")
 					(unit 1)
 				)
@@
 		(dnp no)
 		(fields_autoplaced yes)
-		(property "Reference" "#PWR0105"
+		(property "Reference" "#PWR0106"
 			(at 36.83 90.17 0)
 			(effects
@@
 			(project "Lark"
 				(path "/a351af57-4353-47da-9f45-7393de572768/edc369e3-0a21-4448-a6d2-131219450aa0"
-					(reference "#PWR0105")
+					(reference "#PWR0106")
 					(unit 1)
 				)
@@
 		(dnp no)
 		(fields_autoplaced yes)
-		(property "Reference" "#PWR0112"
+		(property "Reference" "#PWR0113"
 			(at 66.04 186.69 0)
 			(effects
@@
 			(project "Lark"
 				(path "/a351af57-4353-47da-9f45-7393de572768/edc369e3-0a21-4448-a6d2-131219450aa0"
-					(reference "#PWR0112")
+					(reference "#PWR0113")
 					(unit 1)
 				)
@@
 		(dnp no)
 		(fields_autoplaced yes)
-		(property "Reference" "D8"
+		(property "Reference" "D10"
 			(at 40.64 95.5674 90)
 			(effects
@@
 			(project "Lark"
 				(path "/a351af57-4353-47da-9f45-7393de572768/edc369e3-0a21-4448-a6d2-131219450aa0"
-					(reference "D8")
+					(reference "D10")
 					(unit 1)
 				)
@@
 		(dnp no)
 		(fields_autoplaced yes)
-		(property "Reference" "#PWR0108"
+		(property "Reference" "#PWR0109"
 			(at 26.67 156.21 0)
 			(effects
@@
 			(project "Lark"
 				(path "/a351af57-4353-47da-9f45-7393de572768/edc369e3-0a21-4448-a6d2-131219450aa0"
-					(reference "#PWR0108")
+					(reference "#PWR0109")
 					(unit 1)
 				)
@@
 		(on_board yes)
 		(dnp no)
-		(property "Reference" "U11"
+		(property "Reference" "U13"
 			(at 247.65 123.19 0)
 			(effects
@@
 			(project "Lark"
 				(path "/a351af57-4353-47da-9f45-7393de572768/edc369e3-0a21-4448-a6d2-131219450aa0"
-					(reference "U11")
+					(reference "U13")
 					(unit 1)
 				)
@@
 		(dnp no)
 		(fields_autoplaced yes)
-		(property "Reference" "#PWR0106"
+		(property "Reference" "#PWR0107"
 			(at 266.7 125.73 0)
 			(effects
@@
 			(project "Lark"
 				(path "/a351af57-4353-47da-9f45-7393de572768/edc369e3-0a21-4448-a6d2-131219450aa0"
-					(reference "#PWR0106")
-					(unit 1)
-				)
+					(reference "#PWR0107")
+					(unit 1)
+				)

Commit message: Changed revision again...
- It dawned on me that this is rev 2, so the rev is now 01.00.1.
- Added thermal relief to the TH pads so I can actually solder the parts.
- Added more silkscreen to denote the rev, the github link, and ESD sensitivity of the device.
- Made minor pcb changes, I moved a test point, and cleaned up some traces.
Parts:
- U12: now left out of the parts list
