File: Lark/FrontIO.kicad_sch (KiCad schematic)
At the start: 15 parts, among them J4 0530470810

Commit message: added power section to schematic
It needs revised, due to thermal issue. Specifically in regards to my soft start circuit, the mosfet wont be able to handle the power dissipated during a slow turn on.
Parts:
- C18, C19: value 0.1 µF -> 0.1µF
- D10, D11, D12, D8, D9: footprint onsemi:D_SOD-523 -> onsemi:ESD5Z3.3T1G
Connections:
- net +3.3VBC renamed +3.3V
Changed lines of the file:
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@@
 			)
 		)
-		(property "Datasheet" "https://www.seielect.com/catalog/SEI-RMCF_RMCP.pdf"
+		(property "Datasheet" "~"
 			(at 50.8 106.68 0)
 			(effects
@@
 			)
 		)
-		(property "Footprint" "onsemi:D_SOD-523"
+		(property "Footprint" "onsemi:ESD5Z3.3T1G"
 			(at 58.42 173.99 0)
 			(effects
@@
 			)
 		)
-		(property "Footprint" "onsemi:D_SOD-523"
+		(property "Footprint" "onsemi:ESD5Z3.3T1G"
 			(at 59.69 55.88 0)
 			(effects
@@
 			)
 		)
-		(property "Datasheet" "https://www.seielect.com/catalog/SEI-RMCF_RMCP.pdf"
+		(property "Datasheet" "~"
 			(at 80.01 38.1 0)
 			(effects
@@
 			)
 		)
-		(property "Footprint" "onsemi:D_SOD-523"
+		(property "Footprint" "onsemi:ESD5Z3.3T1G"
 			(at 80.01 55.88 0)
 			(effects
@@
 			)
 		)
-		(property "Datasheet" "https://www.seielect.com/catalog/SEI-RMCF_RMCP.pdf"
+		(property "Datasheet" "~"
 			(at 50.8 165.1 0)
 			(effects
@@
 			)
 		)
-		(property "Value" "0.1 µF"
+		(property "Value" "0.1µF"
 			(at 39.37 173.9962 0)
 			(effects
@@
 			)
 		)
-		(property "Datasheet" "https://search.murata.co.jp/Ceramy/image/img/A01X/G101/ENG/GRM188R72A104MA35-01A.pdf"
+		(property "Datasheet" "~"
 			(at 36.83 172.72 0)
 			(effects
@@
 			)
 		)
-		(property "Value" "0.1 µF"
+		(property "Value" "0.1µF"
 			(at 39.37 115.5762 0)
 			(effects
@@
 			)
 		)
-		(property "Datasheet" "https://search.murata.co.jp/Ceramy/image/img/A01X/G101/ENG/GRM188R72A104MA35-01A.pdf"
+		(property "Datasheet" "~"
 			(at 36.83 114.3 0)
 			(effects
@@
 			)
 		)
-		(property "Datasheet" "https://www.seielect.com/catalog/SEI-RMCF_RMCP.pdf"
+		(property "Datasheet" "~"
 			(at 59.69 38.1 0)
 			(effects
@@
 			)
 		)
-		(property "Footprint" "onsemi:D_SOD-523"
+		(property "Footprint" "onsemi:ESD5Z3.3T1G"
 			(at 58.42 115.57 0)
 			(effects
@@
 			)
 		)
-		(property "Value" "+3.3VBC"
+		(property "Value" "+3.3V"
 			(at 36.83 143.51 0)
 			(effects
@@
 			)
 		)
-		(property "Datasheet" "https://www.seielect.com/catalog/SEI-RMCF_RMCP.pdf"
+		(property "Datasheet" "~"
 			(at 38.1 38.1 0)
 			(effects
@@
 			)
 		)
-		(property "Datasheet" "https://www.seielect.com/catalog/SEI-RMCF_RMCP.pdf"
+		(property "Datasheet" "~"
 			(at 36.83 156.21 0)
 			(effects
@@
 			)
 		)
-		(property "Value" "+3.3VBC"
+		(property "Value" "+3.3V"
 			(at 260.35 24.13 0)
 			(effects
@@
 			)
 		)
-		(property "Value" "+3.3VBC"
+		(property "Value" "+3.3V"
 			(at 36.83 85.09 0)
 			(effects
@@
 			)
 		)
-		(property "Footprint" "onsemi:D_SOD-523"
+		(property "Footprint" "onsemi:ESD5Z3.3T1G"
 			(at 38.1 55.88 0)
 			(effects
@@
 			)
 		)
-		(property "Datasheet" "https://www.seielect.com/catalog/SEI-RMCF_RMCP.pdf"
+		(property "Datasheet" "~"
 			(at 36.83 97.79 0)
 			(effects

Commit message: update, WIP
- Reannotated schematic.
- Added STM32 device.
- Fixed High-side switch (removed soft-start cap for device safety).
Parts:
- renumbered C19 to C30, C18 to C31, D9 to D13, D8 to D14, J4 to J5, R38 to R45, R39 to R46, R40 to R47, R36 to R48, R37 to R49, R30 to R50, R35 to R51
Other:
- note added: "Contact Rating 1 Amp Max"
Changed lines of the file:
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@@
+		)
+	)
+	(text "Contact Rating \n1 Amp Max"
+		(exclude_from_sim no)
+		(at 271.78 64.008 0)
+		(effects
+			(font
+				(size 0.762 0.762)
+			)
 		)
 	)
@@
 		(dnp no)
 		(fields_autoplaced yes)
-		(property "Reference" "#PWR094"
+		(property "Reference" "#PWR0139"
 			(at 36.83 129.54 0)
 			(effects
@@
 			(project "Lark"
 				(path "/a351af57-4353-47da-9f45-7393de572768/952214a1-3201-40ca-8c5a-55526392db8f"
-					(reference "#PWR094")
+					(reference "#PWR0139")
 					(unit 1)
 				)
@@
 		(dnp no)
 		(fields_autoplaced yes)
-		(property "Reference" "#PWR0101"
+		(property "Reference" "#PWR0137"
 			(at 80.01 72.39 0)
 			(effects
@@
 			(project "Lark"
 				(path "/a351af57-4353-47da-9f45-7393de572768/952214a1-3201-40ca-8c5a-55526392db8f"
-					(reference "#PWR0101")
+					(reference "#PWR0137")
 					(unit 1)
 				)
@@
 		(on_board yes)
 		(dnp no)
-		(property "Reference" "R37"
+		(property "Reference" "R49"
 			(at 51.816 104.14 90)
 			(effects
@@
 			(project "Lark"
 				(path "/a351af57-4353-47da-9f45-7393de572768/952214a1-3201-40ca-8c5a-55526392db8f"
-					(reference "R37")
+					(reference "R49")
 					(unit 1)
 				)
@@
 		(dnp no)
 		(fields_autoplaced yes)
-		(property "Reference" "#PWR096"
+		(property "Reference" "#PWR0142"
 			(at 36.83 187.96 0)
 			(effects
@@
 			(project "Lark"
 				(path "/a351af57-4353-47da-9f45-7393de572768/952214a1-3201-40ca-8c5a-55526392db8f"
-					(reference "#PWR096")
+					(reference "#PWR0142")
 					(unit 1)
 				)
@@
 		(dnp no)
 		(fields_autoplaced yes)
-		(property "Reference" "D8"
+		(property "Reference" "D14"
 			(at 60.96 173.4501 90)
 			(effects
@@
 			(project "Lark"
 				(path "/a351af57-4353-47da-9f45-7393de572768/952214a1-3201-40ca-8c5a-55526392db8f"
-					(reference "D8")
+					(reference "D14")
 					(unit 1)
 				)
@@
 		(dnp no)
 		(fields_autoplaced yes)
-		(property "Reference" "#PWR098"
+		(property "Reference" "#PWR0140"
 			(at 58.42 129.54 0)
 			(effects
@@
 			(project "Lark"
 				(path "/a351af57-4353-47da-9f45-7393de572768/952214a1-3201-40ca-8c5a-55526392db8f"
-					(reference "#PWR098")
+					(reference "#PWR0140")
 					(unit 1)
 				)
@@
 		(on_board yes)
 		(dnp no)
-		(property "Reference" "R40"
+		(property "Reference" "R47"
 			(at 82.55 36.8299 0)
 			(effects
@@
 			(project "Lark"
 				(path "/a351af57-4353-47da-9f45-7393de572768/952214a1-3201-40ca-8c5a-55526392db8f"
-					(reference "R40")
+					(reference "R47")
 					(unit 1)
 				)
@@
 		(on_board yes)
 		(dnp no)
-		(property "Reference" "R35"
+		(property "Reference" "R51"
 			(at 51.816 162.56 90)
 			(effects
@@
 			(project "Lark"
 				(path "/a351af57-4353-47da-9f45-7393de572768/952214a1-3201-40ca-8c5a-55526392db8f"
-					(reference "R35")
+					(reference "R51")
 					(unit 1)
 				)
@@
 		(on_board yes)
 		(dnp no)
-		(property "Reference" "C18"
+		(property "Reference" "C31"
 			(at 39.37 171.4562 0)
 			(effects
@@
 			(project "Lark"
 				(path "/a351af57-4353-47da-9f45-7393de572768/952214a1-3201-40ca-8c5a-55526392db8f"
-					(reference "C18")
+					(reference "C31")
 					(unit 1)
 				)
@@
 		(on_board yes)
 		(dnp no)
-		(property "Reference" "J4"
+		(property "Reference" "J5"
 			(at 268.478 31.75 0)
 			(effects
@@
 			(project ""
 				(path "/a351af57-4353-47da-9f45-7393de572768/952214a1-3201-40ca-8c5a-55526392db8f"
-					(reference "J4")
+					(reference "J5")
 					(unit 1)
 				)
@@
 		(dnp no)
 		(fields_autoplaced yes)
-		(property "Reference" "#PWR097"
+		(property "Reference" "#PWR0143"
 			(at 58.42 187.96 0)
 			(effects
@@
 			(project "Lark"
 				(path "/a351af57-4353-47da-9f45-7393de572768/952214a1-3201-40ca-8c5a-55526392db8f"
-					(reference "#PWR097")
+					(reference "#PWR0143")
 					(unit 1)
 				)
@@
 		(on_board yes)
 		(dnp no)
-		(property "Reference" "C19"
+		(property "Reference" "C30"
 			(at 39.37 113.0362 0)
 			(effects
@@
 			(project "Lark"
 				(path "/a351af57-4353-47da-9f45-7393de572768/952214a1-3201-40ca-8c5a-55526392db8f"
-					(reference "C19")
+					(reference "C30")
 					(unit 1)
 				)
@@
 		(dnp no)
 		(fields_autoplaced yes)
-		(property "Reference" "#PWR099"
+		(property "Reference" "#PWR0135"
 			(at 38.1 72.39 0)
 			(effects
@@
 			(project "Lark"
 				(path "/a351af57-4353-47da-9f45-7393de572768/952214a1-3201-40ca-8c5a-55526392db8f"
-					(reference "#PWR099")
+					(reference "#PWR0135")
 					(unit 1)
 				)
@@
 		(dnp no)
 		(fields_autoplaced yes)
-		(property "Reference" "#PWR0103"
+		(property "Reference" "#PWR0134"
 			(at 260.35 62.23 0)
 			(effects
@@
 			(project "Lark"
 				(path "/a351af57-4353-47da-9f45-7393de572768/952214a1-3201-40ca-8c5a-55526392db8f"
-					(reference "#PWR0103")
+					(reference "#PWR0134")
 					(unit 1)
 				)
@@
 		(on_board yes)
 		(dnp no)
-		(property "Reference" "R39"
+		(property "Reference" "R46"
 			(at 62.23 36.8299 0)
 			(effects
@@
 			(project "Lark"
 				(path "/a351af57-4353-47da-9f45-7393de572768/952214a1-3201-40ca-8c5a-55526392db8f"
-					(reference "R39")
+					(reference "R46")
 					(unit 1)
 				)
@@
 		(dnp no)
 		(fields_autoplaced yes)
-		(property "Reference" "#PWR0100"
+		(property "Reference" "#PWR0136"
 			(at 59.69 72.39 0)
 			(effects
@@
 			(project "Lark"
 				(path "/a351af57-4353-47da-9f45-7393de572768/952214a1-3201-40ca-8c5a-55526392db8f"
-					(reference "#PWR0100")
+					(reference "#PWR0136")
 					(unit 1)
 				)
@@
 		(dnp no)
 		(fields_autoplaced yes)
-		(property "Reference" "D9"
+		(property "Reference" "D13"
 			(at 60.96 115.0301 90)
 			(effects
@@
 			(project "Lark"
 				(path "/a351af57-4353-47da-9f45-7393de572768/952214a1-3201-40ca-8c5a-55526392db8f"
-					(reference "D9")
+					(reference "D13")
 					(unit 1)
 				)
@@
 		(dnp no)
 		(fields_autoplaced yes)
-		(property "Reference" "#PWR095"
+		(property "Reference" "#PWR0141"
 			(at 36.83 152.4 0)
 			(effects
@@
 			(project "Lark"
 				(path "/a351af57-4353-47da-9f45-7393de572768/952214a1-3201-40ca-8c5a-55526392db8f"
-					(reference "#PWR095")
+					(reference "#PWR0141")
 					(unit 1)
 				)
@@
 		(on_board yes)
 		(dnp no)
-		(property "Reference" "R38"
+		(property "Reference" "R45"
 			(at 40.64 36.8299 0)
 			(effects
@@
 			(project "Lark"
 				(path "/a351af57-4353-47da-9f45-7393de572768/952214a1-3201-40ca-8c5a-55526392db8f"
-					(reference "R38")
+					(reference "R45")
 					(unit 1)
 				)
@@
 		(on_board yes)
 		(dnp no)
-		(property "Reference" "R30"
+		(property "Reference" "R50"
 			(at 39.37 154.9399 0)
 			(effects
@@
 			(project "Lark"
 				(path "/a351af57-4353-47da-9f45-7393de572768/952214a1-3201-40ca-8c5a-55526392db8f"
-					(reference "R30")
+					(reference "R50")
 					(unit 1)
 				)
@@
 		(dnp no)
 		(fields_autoplaced yes)
-		(property "Reference" "#PWR0102"
+		(property "Reference" "#PWR0133"
 			(at 260.35 33.02 0)
 			(effects
@@
 			(project "Lark"
 				(path "/a351af57-4353-47da-9f45-7393de572768/952214a1-3201-40ca-8c5a-55526392db8f"
-					(reference "#PWR0102")
+					(reference "#PWR0133")
 					(unit 1)
 				)
@@
 		(dnp no)
 		(fields_autoplaced yes)
-		(property "Reference" "#PWR093"
+		(property "Reference" "#PWR0138"
 			(at 36.83 93.98 0)
 			(effects
@@
 			(project "Lark"
 				(path "/a351af57-4353-47da-9f45-7393de572768/952214a1-3201-40ca-8c5a-55526392db8f"
-					(reference "#PWR093")
+					(reference "#PWR0138")
 					(unit 1)
 				)
@@
 		(on_board yes)
 		(dnp no)
-		(property "Reference" "R36"
+		(property "Reference" "R48"
 			(at 39.37 96.5199 0)
 			(effects
@@
 			(project "Lark"
 				(path "/a351af57-4353-47da-9f45-7393de572768/952214a1-3201-40ca-8c5a-55526392db8f"
-					(reference "R36")
+					(reference "R48")
 					(unit 1)
 				)

Commit message: Updated schematic, WIP
- Added NOR flash part.
- Added new CubeMX config file.
- Reannotated the schematic.
- Made some more connections to the MCU.
Parts:
- renumbered R45 to R46, R46 to R47, R47 to R48, R48 to R49, R49 to R50, R50 to R51, R51 to R52
Changed lines of the file:
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@@
 		(on_board yes)
 		(dnp no)
-		(property "Reference" "R49"
+		(property "Reference" "R50"
 			(at 51.816 104.14 90)
 			(effects
@@
 			(project "Lark"
 				(path "/a351af57-4353-47da-9f45-7393de572768/952214a1-3201-40ca-8c5a-55526392db8f"
-					(reference "R49")
+					(reference "R50")
 					(unit 1)
 				)
@@
 		(on_board yes)
 		(dnp no)
-		(property "Reference" "R47"
+		(property "Reference" "R48"
 			(at 82.55 36.8299 0)
 			(effects
@@
 			(project "Lark"
 				(path "/a351af57-4353-47da-9f45-7393de572768/952214a1-3201-40ca-8c5a-55526392db8f"
-					(reference "R47")
+					(reference "R48")
 					(unit 1)
 				)
@@
 		(on_board yes)
 		(dnp no)
-		(property "Reference" "R51"
+		(property "Reference" "R52"
 			(at 51.816 162.56 90)
 			(effects
@@
 			(project "Lark"
 				(path "/a351af57-4353-47da-9f45-7393de572768/952214a1-3201-40ca-8c5a-55526392db8f"
-					(reference "R51")
+					(reference "R52")
 					(unit 1)
 				)
@@
 		(on_board yes)
 		(dnp no)
-		(property "Reference" "R46"
+		(property "Reference" "R47"
 			(at 62.23 36.8299 0)
 			(effects
@@
 			(project "Lark"
 				(path "/a351af57-4353-47da-9f45-7393de572768/952214a1-3201-40ca-8c5a-55526392db8f"
-					(reference "R46")
+					(reference "R47")
 					(unit 1)
 				)
@@
 		(on_board yes)
 		(dnp no)
-		(property "Reference" "R45"
+		(property "Reference" "R46"
 			(at 40.64 36.8299 0)
 			(effects
@@
 			(project "Lark"
 				(path "/a351af57-4353-47da-9f45-7393de572768/952214a1-3201-40ca-8c5a-55526392db8f"
-					(reference "R45")
+					(reference "R46")
 					(unit 1)
 				)
@@
 		(on_board yes)
 		(dnp no)
-		(property "Reference" "R50"
+		(property "Reference" "R51"
 			(at 39.37 154.9399 0)
 			(effects
@@
 			(project "Lark"
 				(path "/a351af57-4353-47da-9f45-7393de572768/952214a1-3201-40ca-8c5a-55526392db8f"
-					(reference "R50")
+					(reference "R51")
 					(unit 1)
 				)
@@
 		(on_board yes)
 		(dnp no)
-		(property "Reference" "R48"
+		(property "Reference" "R49"
 			(at 39.37 96.5199 0)
 			(effects
@@
 			(project "Lark"
 				(path "/a351af57-4353-47da-9f45-7393de572768/952214a1-3201-40ca-8c5a-55526392db8f"
-					(reference "R48")
-					(unit 1)
-				)
+					(reference "R49")
+					(unit 1)
+				)

Commit message: Update, WIP
- Added TVS diode to 24v Supply.
- Fixed bleeder circuit at some point (I think it was this commit)
- Added Jumper to connect NTC to ADC. (again I think it was this commit)
Parts:
- renumbered D10 to D11, D11 to D12, D12 to D13, D13 to D14, D14 to D15, R46 to R49, R47 to R50, R48 to R51, R49 to R52, R50 to R53, R51 to R54, R52 to R55
Changed lines of the file:
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@@
 		(dnp no)
 		(fields_autoplaced yes)
-		(property "Reference" "#PWR0139"
+		(property "Reference" "#PWR0143"
 			(at 36.83 129.54 0)
 			(effects
@@
 			(project "Lark"
 				(path "/a351af57-4353-47da-9f45-7393de572768/952214a1-3201-40ca-8c5a-55526392db8f"
-					(reference "#PWR0139")
+					(reference "#PWR0143")
 					(unit 1)
 				)
@@
 		(dnp no)
 		(fields_autoplaced yes)
-		(property "Reference" "#PWR0137"
+		(property "Reference" "#PWR0141"
 			(at 80.01 72.39 0)
 			(effects
@@
 			(project "Lark"
 				(path "/a351af57-4353-47da-9f45-7393de572768/952214a1-3201-40ca-8c5a-55526392db8f"
-					(reference "#PWR0137")
+					(reference "#PWR0141")
 					(unit 1)
 				)
@@
 		(on_board yes)
 		(dnp no)
-		(property "Reference" "R50"
+		(property "Reference" "R53"
 			(at 51.816 104.14 90)
 			(effects
@@
 			(project "Lark"
 				(path "/a351af57-4353-47da-9f45-7393de572768/952214a1-3201-40ca-8c5a-55526392db8f"
-					(reference "R50")
+					(reference "R53")
 					(unit 1)
 				)
@@
 		(dnp no)
 		(fields_autoplaced yes)
-		(property "Reference" "#PWR0142"
+		(property "Reference" "#PWR0146"
 			(at 36.83 187.96 0)
 			(effects
@@
 			(project "Lark"
 				(path "/a351af57-4353-47da-9f45-7393de572768/952214a1-3201-40ca-8c5a-55526392db8f"
-					(reference "#PWR0142")
+					(reference "#PWR0146")
 					(unit 1)
 				)
@@
 		(dnp no)
 		(fields_autoplaced yes)
-		(property "Reference" "D14"
+		(property "Reference" "D15"
 			(at 60.96 173.4501 90)
 			(effects
@@
 			(project "Lark"
 				(path "/a351af57-4353-47da-9f45-7393de572768/952214a1-3201-40ca-8c5a-55526392db8f"
-					(reference "D14")
+					(reference "D15")
 					(unit 1)
 				)
@@
 		(dnp no)
 		(fields_autoplaced yes)
-		(property "Reference" "D11"
+		(property "Reference" "D12"
 			(at 62.23 55.3401 90)
 			(effects
@@
 			(project "Lark"
 				(path "/a351af57-4353-47da-9f45-7393de572768/952214a1-3201-40ca-8c5a-55526392db8f"
-					(reference "D11")
+					(reference "D12")
 					(unit 1)
 				)
@@
 		(dnp no)
 		(fields_autoplaced yes)
-		(property "Reference" "#PWR0140"
+		(property "Reference" "#PWR0144"
 			(at 58.42 129.54 0)
 			(effects
@@
 			(project "Lark"
 				(path "/a351af57-4353-47da-9f45-7393de572768/952214a1-3201-40ca-8c5a-55526392db8f"
-					(reference "#PWR0140")
+					(reference "#PWR0144")
 					(unit 1)
 				)
@@
 		(on_board yes)
 		(dnp no)
-		(property "Reference" "R48"
+		(property "Reference" "R51"
 			(at 82.55 36.8299 0)
 			(effects
@@
 			(project "Lark"
 				(path "/a351af57-4353-47da-9f45-7393de572768/952214a1-3201-40ca-8c5a-55526392db8f"
-					(reference "R48")
+					(reference "R51")
 					(unit 1)
 				)
@@
 		(dnp no)
 		(fields_autoplaced yes)
-		(property "Reference" "D12"
+		(property "Reference" "D13"
 			(at 82.55 55.3401 90)
 			(effects
@@
 			(project "Lark"
 				(path "/a351af57-4353-47da-9f45-7393de572768/952214a1-3201-40ca-8c5a-55526392db8f"
-					(reference "D12")
+					(reference "D13")
 					(unit 1)
 				)
@@
 		(on_board yes)
 		(dnp no)
-		(property "Reference" "R52"
+		(property "Reference" "R55"
 			(at 51.816 162.56 90)
 			(effects
@@
 			(project "Lark"
 				(path "/a351af57-4353-47da-9f45-7393de572768/952214a1-3201-40ca-8c5a-55526392db8f"
-					(reference "R52")
+					(reference "R55")
 					(unit 1)
 				)
@@
 		(dnp no)
 		(fields_autoplaced yes)
-		(property "Reference" "#PWR0143"
+		(property "Reference" "#PWR0147"
 			(at 58.42 187.96 0)
 			(effects
@@
 			(project "Lark"
 				(path "/a351af57-4353-47da-9f45-7393de572768/952214a1-3201-40ca-8c5a-55526392db8f"
-					(reference "#PWR0143")
+					(reference "#PWR0147")
 					(unit 1)
 				)
@@
 		(dnp no)
 		(fields_autoplaced yes)
-		(property "Reference" "#PWR0135"
+		(property "Reference" "#PWR0139"
 			(at 38.1 72.39 0)
 			(effects
@@
 			(project "Lark"
 				(path "/a351af57-4353-47da-9f45-7393de572768/952214a1-3201-40ca-8c5a-55526392db8f"
-					(reference "#PWR0135")
+					(reference "#PWR0139")
 					(unit 1)
 				)
@@
 		(dnp no)
 		(fields_autoplaced yes)
-		(property "Reference" "#PWR0134"
+		(property "Reference" "#PWR0138"
 			(at 260.35 62.23 0)
 			(effects
@@
 			(project "Lark"
 				(path "/a351af57-4353-47da-9f45-7393de572768/952214a1-3201-40ca-8c5a-55526392db8f"
-					(reference "#PWR0134")
+					(reference "#PWR0138")
 					(unit 1)
 				)
@@
 		(on_board yes)
 		(dnp no)
-		(property "Reference" "R47"
+		(property "Reference" "R50"
 			(at 62.23 36.8299 0)
 			(effects
@@
 			(project "Lark"
 				(path "/a351af57-4353-47da-9f45-7393de572768/952214a1-3201-40ca-8c5a-55526392db8f"
-					(reference "R47")
+					(reference "R50")
 					(unit 1)
 				)
@@
 		(dnp no)
 		(fields_autoplaced yes)
-		(property "Reference" "#PWR0136"
+		(property "Reference" "#PWR0140"
 			(at 59.69 72.39 0)
 			(effects
@@
 			(project "Lark"
 				(path "/a351af57-4353-47da-9f45-7393de572768/952214a1-3201-40ca-8c5a-55526392db8f"
-					(reference "#PWR0136")
+					(reference "#PWR0140")
 					(unit 1)
 				)
@@
 		(dnp no)
 		(fields_autoplaced yes)
-		(property "Reference" "D13"
+		(property "Reference" "D14"
 			(at 60.96 115.0301 90)
 			(effects
@@
 			(project "Lark"
 				(path "/a351af57-4353-47da-9f45-7393de572768/952214a1-3201-40ca-8c5a-55526392db8f"
-					(reference "D13")
+					(reference "D14")
 					(unit 1)
 				)
@@
 		(dnp no)
 		(fields_autoplaced yes)
-		(property "Reference" "#PWR0141"
+		(property "Reference" "#PWR0145"
 			(at 36.83 152.4 0)
 			(effects
@@
 			(project "Lark"
 				(path "/a351af57-4353-47da-9f45-7393de572768/952214a1-3201-40ca-8c5a-55526392db8f"
-					(reference "#PWR0141")
+					(reference "#PWR0145")
 					(unit 1)
 				)
@@
 		(on_board yes)
 		(dnp no)
-		(property "Reference" "R46"
+		(property "Reference" "R49"
 			(at 40.64 36.8299 0)
 			(effects
@@
 			(project "Lark"
 				(path "/a351af57-4353-47da-9f45-7393de572768/952214a1-3201-40ca-8c5a-55526392db8f"
-					(reference "R46")
+					(reference "R49")
 					(unit 1)
 				)
@@
 		(on_board yes)
 		(dnp no)
-		(property "Reference" "R51"
+		(property "Reference" "R54"
 			(at 39.37 154.9399 0)
 			(effects
@@
 			(project "Lark"
 				(path "/a351af57-4353-47da-9f45-7393de572768/952214a1-3201-40ca-8c5a-55526392db8f"
-					(reference "R51")
+					(reference "R54")
 					(unit 1)
 				)
@@
 		(dnp no)
 		(fields_autoplaced yes)
-		(property "Reference" "#PWR0133"
+		(property "Reference" "#PWR0137"
 			(at 260.35 33.02 0)
 			(effects
@@
 			(project "Lark"
 				(path "/a351af57-4353-47da-9f45-7393de572768/952214a1-3201-40ca-8c5a-55526392db8f"
-					(reference "#PWR0133")
+					(reference "#PWR0137")
 					(unit 1)
 				)
@@
 		(dnp no)
 		(fields_autoplaced yes)
-		(property "Reference" "#PWR0138"
+		(property "Reference" "#PWR0142"
 			(at 36.83 93.98 0)
 			(effects
@@
 			(project "Lark"
 				(path "/a351af57-4353-47da-9f45-7393de572768/952214a1-3201-40ca-8c5a-55526392db8f"
-					(reference "#PWR0138")
+					(reference "#PWR0142")
 					(unit 1)
 				)
@@
 		(dnp no)
 		(fields_autoplaced yes)
-		(property "Reference" "D10"
+		(property "Reference" "D11"
 			(at 40.64 55.3401 90)
 			(effects
@@
 			(project "Lark"
 				(path "/a351af57-4353-47da-9f45-7393de572768/952214a1-3201-40ca-8c5a-55526392db8f"
-					(reference "D10")
+					(reference "D11")
 					(unit 1)
 				)
@@
 		(on_board yes)
 		(dnp no)
-		(property "Reference" "R49"
+		(property "Reference" "R52"
 			(at 39.37 96.5199 0)
 			(effects
@@
 			(project "Lark"
 				(path "/a351af57-4353-47da-9f45-7393de572768/952214a1-3201-40ca-8c5a-55526392db8f"
-					(reference "R49")
-					(unit 1)
-				)
+					(reference "R52")
+					(unit 1)
+				)

Commit message: updated WIP
- fixed high-side switch (swapped out pfets)
- swapped out bleeder fet.
- changed a few footprints.
- changed zeners to 15v ones
- added soft-start cap back in to the high-side switch.

(today ive mainly been struggling with the inrush current, but I think its solved now)
Parts:
- renumbered C30 to C31, C31 to C32, D11 to D13, D12 to D14, D13 to D15, D14 to D16, D15 to D17
Other:
- note added: "LED: QBLP600-RGB5-3164"

Commit message: started on layout, WIP
I'm not a fan of how its going, I feel like I might redo it, before I get to far into it. A patchy foundation makes an unstable house.
Connections:
- net BTN_1: now also D17.1 (Cathode), R55.2
- net BTN_2: no longer D17.1 (Cathode), R55.2
Changed lines of the file:
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@@
 		)
 	)
-	(label "BTN_2"
+	(label "BTN_1"
 		(at 66.04 165.1 180)
 		(effects
