File: Lark/Motor_Driver.kicad_sch (KiCad schematic)
At the start: 13 parts, among them U5 A4985SESTR-T

Commit message: still porting design over from 'other' cad software.
Parts:
- added C11: 100 µF, Panasonic Electronic Components:ECA-1VM101, symbol Panasonic Electronic Components:ECA-1VM101
- TP7: footprint (none) -> TestPoint:TestPoint_Pad_D1.0mm
Connections:
- net +24V: now also C11.1
- net GND: now also C11.2
Other:
- note added: "Bulk Cap"
- note added: "Test Points"
- moved on the sheet: TP7

Commit message: added power section to schematic
It needs revised, due to thermal issue. Specifically in regards to my soft start circuit, the mosfet wont be able to handle the power dissipated during a slow turn on.
Parts:
- C10, C5, C6, C8, C9: value 0.1 µF -> 0.1µF
- C11: value 100 µF -> 100µF
- C7: value 0.22 µF -> 0.22µF
Changed lines of the file:
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@@
 			)
 		)
-		(property "Value" "0.22 µF"
+		(property "Value" "0.22µF"
 			(at 248.92 146.0562 0)
 			(effects
@@
 			)
 		)
-		(property "Datasheet" "https://search.murata.co.jp/Ceramy/image/img/A01X/G101/ENG/GRM188R71H224KAC4-01.pdf"
+		(property "Datasheet" "~"
 			(at 246.38 144.78 0)
 			(effects
@@
 			)
 		)
-		(property "Datasheet" "https://www.seielect.com/catalog/SEI-RMCF_RMCP.pdf"
+		(property "Datasheet" "~"
 			(at 118.11 67.31 0)
 			(effects
@@
 			)
 		)
-		(property "Value" "100 µF"
+		(property "Value" "100µF"
 			(at 88.9 175.6409 0)
 			(effects
@@
 			)
 		)
-		(property "Datasheet" "https://www.seielect.com/catalog/SEI-CSR_CSRN.pdf"
+		(property "Datasheet" "~"
 			(at 259.08 144.78 0)
 			(effects
@@
 			)
 		)
-		(property "Value" "0.1 µF"
+		(property "Value" "0.1µF"
 			(at 26.67 176.5362 0)
 			(effects
@@
 			)
 		)
-		(property "Datasheet" "https://search.murata.co.jp/Ceramy/image/img/A01X/G101/ENG/GRM188R72A104MA35-01A.pdf"
+		(property "Datasheet" "~"
 			(at 24.13 175.26 0)
 			(effects
@@
 			)
 		)
-		(property "Value" "0.1 µF"
+		(property "Value" "0.1µF"
 			(at 273.05 110.4962 0)
 			(effects
@@
 			)
 		)
-		(property "Datasheet" "https://search.murata.co.jp/Ceramy/image/img/A01X/G101/ENG/GRM188R72A104MA35-01A.pdf"
+		(property "Datasheet" "~"
 			(at 270.51 109.22 0)
 			(effects
@@
 			)
 		)
-		(property "Datasheet" "https://www.seielect.com/catalog/SEI-RMCF_RMCP.pdf"
+		(property "Datasheet" "~"
 			(at 233.68 144.78 0)
 			(effects
@@
 			)
 		)
-		(property "Datasheet" "https://www.seielect.com/catalog/SEI-CSR_CSRN.pdf"
+		(property "Datasheet" "~"
 			(at 270.51 144.78 0)
 			(effects
@@
 			)
 		)
-		(property "Value" "0.1 µF"
+		(property "Value" "0.1µF"
 			(at 260.35 110.4962 0)
 			(effects
@@
 			)
 		)
-		(property "Datasheet" "https://search.murata.co.jp/Ceramy/image/img/A01X/G101/ENG/GRM188R72A104MA35-01A.pdf"
+		(property "Datasheet" "~"
 			(at 257.81 109.22 0)
 			(effects
@@
 			)
 		)
-		(property "Datasheet" "https://www.seielect.com/catalog/SEI-RMCF_RMCP.pdf"
+		(property "Datasheet" "~"
 			(at 223.52 144.78 0)
 			(effects
@@
 			)
 		)
-		(property "Value" "0.1 µF"
+		(property "Value" "0.1µF"
 			(at 40.64 176.5362 0)
 			(effects
@@
 			)
 		)
-		(property "Datasheet" "https://search.murata.co.jp/Ceramy/image/img/A01X/G101/ENG/GRM188R72A104MA35-01A.pdf"
+		(property "Datasheet" "~"
 			(at 38.1 175.26 0)
 			(effects
@@
 			)
 		)
-		(property "Value" "0.1 µF"
+		(property "Value" "0.1µF"
 			(at 55.88 176.5362 0)
 			(effects
@@
 			)
 		)
-		(property "Datasheet" "https://search.murata.co.jp/Ceramy/image/img/A01X/G101/ENG/GRM188R72A104MA35-01A.pdf"
+		(property "Datasheet" "~"
 			(at 53.34 175.26 0)
 			(effects

Commit message: update, WIP
- Reannotated schematic.
- Added STM32 device.
- Fixed High-side switch (removed soft-start cap for device safety).
Parts:
- renumbered C5 to C17, C6 to C18, C7 to C19, C8 to C20, C9 to C21, C10 to C22, C11 to C23, R19 to R30, R20 to R31, R21 to R32, R22 to R33, R23 to R34, TP7 to TP12, U5 to U8

Commit message: Updated schematic, WIP
- Added NOR flash part.
- Added new CubeMX config file.
- Reannotated the schematic.
- Made some more connections to the MCU.
Parts:
- renumbered R30 to R31, R31 to R32, R32 to R33, R33 to R34, R34 to R35
Other:
- moved on the sheet: TP12
Changed lines of the file:
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@@
 	)
 	(rectangle
-		(start 251.46 19.05)
-		(end 280.67 35.56)
+		(start 15.24 130.81)
+		(end 34.29 147.32)
 		(stroke
 			(width 0)
@@
 	(text "Test Points"
 		(exclude_from_sim no)
-		(at 251.206 17.526 0)
+		(at 14.986 129.286 0)
 		(effects
 			(font
@@
 	(wire
 		(pts
-			(xy 266.7 26.67) (xy 266.7 31.75)
+			(xy 20.32 138.43) (xy 20.32 143.51)
 		)
 		(stroke
@@
 	(wire
 		(pts
-			(xy 259.08 31.75) (xy 266.7 31.75)
+			(xy 26.67 143.51) (xy 20.32 143.51)
 		)
 		(stroke
@@
 	)
 	(label "VREF"
-		(at 259.08 31.75 0)
+		(at 26.67 143.51 180)
 		(effects
 			(font
 				(size 1.27 1.27)
 			)
-			(justify left bottom)
+			(justify right bottom)
 		)
 	)
@@
 		(on_board yes)
 		(dnp no)
-		(property "Reference" "R30"
+		(property "Reference" "R31"
 			(at 120.65 66.0399 0)
 			(effects
@@
 			(project "Lark"
 				(path "/a351af57-4353-47da-9f45-7393de572768/4f6e6a31-1617-4951-bb1f-ffce39c005db"
-					(reference "R30")
+					(reference "R31")
 					(unit 1)
 				)
@@
 	(symbol
 		(lib_id "Connector:TestPoint")
-		(at 266.7 26.67 0)
+		(at 20.32 138.43 0)
 		(unit 1)
 		(exclude_from_sim no)
@@
 		(fields_autoplaced yes)
 		(property "Reference" "TP12"
-			(at 269.24 22.0979 0)
+			(at 22.86 133.8579 0)
 			(effects
 				(font
@@
 		)
 		(property "Value" "TestPoint"
-			(at 269.24 24.6379 0)
+			(at 22.86 136.3979 0)
 			(effects
 				(font
@@
 		)
 		(property "Footprint" "TestPoint:TestPoint_Pad_D1.0mm"
-			(at 271.78 26.67 0)
+			(at 25.4 138.43 0)
 			(effects
 				(font
@@
 		)
 		(property "Datasheet" "~"
-			(at 271.78 26.67 0)
+			(at 25.4 138.43 0)
 			(effects
 				(font
@@
 		)
 		(property "Description" "test point"
-			(at 266.7 26.67 0)
+			(at 20.32 138.43 0)
 			(effects
 				(font
@@
 		(on_board yes)
 		(dnp no)
-		(property "Reference" "R33"
+		(property "Reference" "R34"
 			(at 261.62 143.5099 0)
 			(effects
@@
 			(project "Lark"
 				(path "/a351af57-4353-47da-9f45-7393de572768/4f6e6a31-1617-4951-bb1f-ffce39c005db"
-					(reference "R33")
+					(reference "R34")
 					(unit 1)
 				)
@@
 		(on_board yes)
 		(dnp no)
-		(property "Reference" "R32"
+		(property "Reference" "R33"
 			(at 236.22 143.5099 0)
 			(effects
@@
 			(project "Lark"
 				(path "/a351af57-4353-47da-9f45-7393de572768/4f6e6a31-1617-4951-bb1f-ffce39c005db"
-					(reference "R32")
+					(reference "R33")
 					(unit 1)
 				)
@@
 		(on_board yes)
 		(dnp no)
-		(property "Reference" "R34"
+		(property "Reference" "R35"
 			(at 273.05 143.5099 0)
 			(effects
@@
 			(project "Lark"
 				(path "/a351af57-4353-47da-9f45-7393de572768/4f6e6a31-1617-4951-bb1f-ffce39c005db"
-					(reference "R34")
+					(reference "R35")
 					(unit 1)
 				)
@@
 		(on_board yes)
 		(dnp no)
-		(property "Reference" "R31"
+		(property "Reference" "R32"
 			(at 226.06 143.5099 0)
 			(effects
@@
 			(project "Lark"
 				(path "/a351af57-4353-47da-9f45-7393de572768/4f6e6a31-1617-4951-bb1f-ffce39c005db"
-					(reference "R31")
+					(reference "R32")
 					(unit 1)
 				)

Commit message: Update, WIP
- Added TVS diode to 24v Supply.
- Fixed bleeder circuit at some point (I think it was this commit)
- Added Jumper to connect NTC to ADC. (again I think it was this commit)
Parts:
- renumbered R31 to R34, R32 to R35, R33 to R36, R34 to R37, R35 to R38
Changed lines of the file:
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@@
 		(dnp no)
 		(fields_autoplaced yes)
-		(property "Reference" "#PWR077"
+		(property "Reference" "#PWR081"
 			(at 172.72 63.5 0)
 			(effects
@@
 			(project "Lark"
 				(path "/a351af57-4353-47da-9f45-7393de572768/4f6e6a31-1617-4951-bb1f-ffce39c005db"
-					(reference "#PWR077")
+					(reference "#PWR081")
 					(unit 1)
 				)
@@
 		(on_board yes)
 		(dnp no)
-		(property "Reference" "R31"
+		(property "Reference" "R34"
 			(at 120.65 66.0399 0)
 			(effects
@@
 			(project "Lark"
 				(path "/a351af57-4353-47da-9f45-7393de572768/4f6e6a31-1617-4951-bb1f-ffce39c005db"
-					(reference "R31")
+					(reference "R34")
 					(unit 1)
 				)
@@
 		(dnp no)
 		(fields_autoplaced yes)
-		(property "Reference" "#PWR076"
+		(property "Reference" "#PWR080"
 			(at 128.27 63.5 0)
 			(effects
@@
 			(project "Lark"
 				(path "/a351af57-4353-47da-9f45-7393de572768/4f6e6a31-1617-4951-bb1f-ffce39c005db"
-					(reference "#PWR076")
+					(reference "#PWR080")
 					(unit 1)
 				)
@@
 		(dnp no)
 		(fields_autoplaced yes)
-		(property "Reference" "#PWR083"
+		(property "Reference" "#PWR087"
 			(at 259.08 161.29 0)
 			(effects
@@
 			(project "Lark"
 				(path "/a351af57-4353-47da-9f45-7393de572768/4f6e6a31-1617-4951-bb1f-ffce39c005db"
-					(reference "#PWR083")
+					(reference "#PWR087")
 					(unit 1)
 				)
@@
 		(dnp no)
 		(fields_autoplaced yes)
-		(property "Reference" "#PWR085"
+		(property "Reference" "#PWR089"
 			(at 24.13 170.18 0)
 			(effects
@@
 			(project "Lark"
 				(path "/a351af57-4353-47da-9f45-7393de572768/4f6e6a31-1617-4951-bb1f-ffce39c005db"
-					(reference "#PWR085")
+					(reference "#PWR089")
 					(unit 1)
 				)
@@
 		(on_board yes)
 		(dnp no)
-		(property "Reference" "R34"
+		(property "Reference" "R37"
 			(at 261.62 143.5099 0)
 			(effects
@@
 			(project "Lark"
 				(path "/a351af57-4353-47da-9f45-7393de572768/4f6e6a31-1617-4951-bb1f-ffce39c005db"
-					(reference "R34")
+					(reference "R37")
 					(unit 1)
 				)
@@
 		(dnp no)
 		(fields_autoplaced yes)
-		(property "Reference" "#PWR091"
+		(property "Reference" "#PWR095"
 			(at 85.09 191.77 0)
 			(effects
@@
 			(project "Lark"
 				(path "/a351af57-4353-47da-9f45-7393de572768/4f6e6a31-1617-4951-bb1f-ffce39c005db"
-					(reference "#PWR091")
+					(reference "#PWR095")
 					(unit 1)
 				)
@@
 		(dnp no)
 		(fields_autoplaced yes)
-		(property "Reference" "#PWR086"
+		(property "Reference" "#PWR090"
 			(at 53.34 170.18 0)
 			(effects
@@
 			(project "Lark"
 				(path "/a351af57-4353-47da-9f45-7393de572768/4f6e6a31-1617-4951-bb1f-ffce39c005db"
-					(reference "#PWR086")
+					(reference "#PWR090")
 					(unit 1)
 				)
@@
 		(dnp no)
 		(fields_autoplaced yes)
-		(property "Reference" "#PWR078"
+		(property "Reference" "#PWR082"
 			(at 270.51 104.14 0)
 			(effects
@@
 			(project "Lark"
 				(path "/a351af57-4353-47da-9f45-7393de572768/4f6e6a31-1617-4951-bb1f-ffce39c005db"
-					(reference "#PWR078")
+					(reference "#PWR082")
 					(unit 1)
 				)
@@
 		(dnp no)
 		(fields_autoplaced yes)
-		(property "Reference" "#PWR090"
+		(property "Reference" "#PWR094"
 			(at 53.34 191.77 0)
 			(effects
@@
 			(project "Lark"
 				(path "/a351af57-4353-47da-9f45-7393de572768/4f6e6a31-1617-4951-bb1f-ffce39c005db"
-					(reference "#PWR090")
+					(reference "#PWR094")
 					(unit 1)
 				)
@@
 		(dnp no)
 		(fields_autoplaced yes)
-		(property "Reference" "#PWR087"
+		(property "Reference" "#PWR091"
 			(at 85.09 170.18 0)
 			(effects
@@
 			(project "Lark"
 				(path "/a351af57-4353-47da-9f45-7393de572768/4f6e6a31-1617-4951-bb1f-ffce39c005db"
-					(reference "#PWR087")
+					(reference "#PWR091")
 					(unit 1)
 				)
@@
 		(dnp no)
 		(fields_autoplaced yes)
-		(property "Reference" "#PWR089"
+		(property "Reference" "#PWR093"
 			(at 38.1 191.77 0)
 			(effects
@@
 			(project "Lark"
 				(path "/a351af57-4353-47da-9f45-7393de572768/4f6e6a31-1617-4951-bb1f-ffce39c005db"
-					(reference "#PWR089")
+					(reference "#PWR093")
 					(unit 1)
 				)
@@
 		(dnp no)
 		(fields_autoplaced yes)
-		(property "Reference" "#PWR088"
+		(property "Reference" "#PWR092"
 			(at 24.13 191.77 0)
 			(effects
@@
 			(project "Lark"
 				(path "/a351af57-4353-47da-9f45-7393de572768/4f6e6a31-1617-4951-bb1f-ffce39c005db"
-					(reference "#PWR088")
+					(reference "#PWR092")
 					(unit 1)
 				)
@@
 		(dnp no)
 		(fields_autoplaced yes)
-		(property "Reference" "#PWR079"
+		(property "Reference" "#PWR083"
 			(at 163.83 119.38 0)
 			(effects
@@
 			(project "Lark"
 				(path "/a351af57-4353-47da-9f45-7393de572768/4f6e6a31-1617-4951-bb1f-ffce39c005db"
-					(reference "#PWR079")
+					(reference "#PWR083")
 					(unit 1)
 				)
@@
 		(dnp no)
 		(fields_autoplaced yes)
-		(property "Reference" "#PWR084"
+		(property "Reference" "#PWR088"
 			(at 270.51 161.29 0)
 			(effects
@@
 			(project "Lark"
 				(path "/a351af57-4353-47da-9f45-7393de572768/4f6e6a31-1617-4951-bb1f-ffce39c005db"
-					(reference "#PWR084")
+					(reference "#PWR088")
 					(unit 1)
 				)
@@
 		(dnp no)
 		(fields_autoplaced yes)
-		(property "Reference" "#PWR075"
+		(property "Reference" "#PWR079"
 			(at 118.11 63.5 0)
 			(effects
@@
 			(project "Lark"
 				(path "/a351af57-4353-47da-9f45-7393de572768/4f6e6a31-1617-4951-bb1f-ffce39c005db"
-					(reference "#PWR075")
+					(reference "#PWR079")
 					(unit 1)
 				)
@@
 		(on_board yes)
 		(dnp no)
-		(property "Reference" "R33"
+		(property "Reference" "R36"
 			(at 236.22 143.5099 0)
 			(effects
@@
 			(project "Lark"
 				(path "/a351af57-4353-47da-9f45-7393de572768/4f6e6a31-1617-4951-bb1f-ffce39c005db"
-					(reference "R33")
+					(reference "R36")
 					(unit 1)
 				)
@@
 		(dnp no)
 		(fields_autoplaced yes)
-		(property "Reference" "#PWR081"
+		(property "Reference" "#PWR085"
 			(at 233.68 161.29 0)
 			(effects
@@
 			(project "Lark"
 				(path "/a351af57-4353-47da-9f45-7393de572768/4f6e6a31-1617-4951-bb1f-ffce39c005db"
-					(reference "#PWR081")
+					(reference "#PWR085")
 					(unit 1)
 				)
@@
 		(dnp no)
 		(fields_autoplaced yes)
-		(property "Reference" "#PWR080"
+		(property "Reference" "#PWR084"
 			(at 223.52 161.29 0)
 			(effects
@@
 			(project "Lark"
 				(path "/a351af57-4353-47da-9f45-7393de572768/4f6e6a31-1617-4951-bb1f-ffce39c005db"
-					(reference "#PWR080")
+					(reference "#PWR084")
 					(unit 1)
 				)
@@
 		(dnp no)
 		(fields_autoplaced yes)
-		(property "Reference" "#PWR082"
+		(property "Reference" "#PWR086"
 			(at 246.38 161.29 0)
 			(effects
@@
 			(project "Lark"
 				(path "/a351af57-4353-47da-9f45-7393de572768/4f6e6a31-1617-4951-bb1f-ffce39c005db"
-					(reference "#PWR082")
+					(reference "#PWR086")
 					(unit 1)
 				)
@@
 		(on_board yes)
 		(dnp no)
-		(property "Reference" "R35"
+		(property "Reference" "R38"
 			(at 273.05 143.5099 0)
 			(effects
@@
 			(project "Lark"
 				(path "/a351af57-4353-47da-9f45-7393de572768/4f6e6a31-1617-4951-bb1f-ffce39c005db"
-					(reference "R35")
+					(reference "R38")
 					(unit 1)
 				)
@@
 		(on_board yes)
 		(dnp no)
-		(property "Reference" "R32"
+		(property "Reference" "R35"
 			(at 226.06 143.5099 0)
 			(effects
@@
 			(project "Lark"
 				(path "/a351af57-4353-47da-9f45-7393de572768/4f6e6a31-1617-4951-bb1f-ffce39c005db"
-					(reference "R32")
-					(unit 1)
-				)
+					(reference "R35")
+					(unit 1)
+				)
