File: Lark/Motor_Driver.kicad_sch (KiCad schematic)
At the start: 14 parts, among them U8 A4985SESTR-T

Commit message: updated WIP
- fixed high-side switch (swapped out pfets)
- swapped out bleeder fet.
- changed a few footprints.
- changed zeners to 15v ones
- added soft-start cap back in to the high-side switch.

(today ive mainly been struggling with the inrush current, but I think its solved now)
Parts:
- renumbered C17 to C18, C18 to C19, C19 to C20, C20 to C21, C21 to C22, C22 to C23, C23 to C24, U8 to U10
Changed lines of the file:
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@@
 		(on_board yes)
 		(dnp no)
-		(property "Reference" "C19"
+		(property "Reference" "C20"
 			(at 248.92 143.5162 0)
 			(effects
@@
 			(project "Lark"
 				(path "/a351af57-4353-47da-9f45-7393de572768/4f6e6a31-1617-4951-bb1f-ffce39c005db"
-					(reference "C19")
+					(reference "C20")
 					(unit 1)
 				)
@@
 		(dnp no)
 		(fields_autoplaced yes)
-		(property "Reference" "#PWR081"
+		(property "Reference" "#PWR082"
 			(at 172.72 63.5 0)
 			(effects
@@
 			(project "Lark"
 				(path "/a351af57-4353-47da-9f45-7393de572768/4f6e6a31-1617-4951-bb1f-ffce39c005db"
-					(reference "#PWR081")
+					(reference "#PWR082")
 					(unit 1)
 				)
@@
 		(dnp no)
 		(fields_autoplaced yes)
-		(property "Reference" "#PWR080"
+		(property "Reference" "#PWR081"
 			(at 128.27 63.5 0)
 			(effects
@@
 			(project "Lark"
 				(path "/a351af57-4353-47da-9f45-7393de572768/4f6e6a31-1617-4951-bb1f-ffce39c005db"
-					(reference "#PWR080")
+					(reference "#PWR081")
 					(unit 1)
 				)
@@
 		(dnp no)
 		(fields_autoplaced yes)
-		(property "Reference" "C23"
+		(property "Reference" "C24"
 			(at 88.9 173.1009 0)
 			(effects
@@
 			(project "Lark"
 				(path "/a351af57-4353-47da-9f45-7393de572768/4f6e6a31-1617-4951-bb1f-ffce39c005db"
-					(reference "C23")
+					(reference "C24")
 					(unit 1)
 				)
@@
 		(dnp no)
 		(fields_autoplaced yes)
-		(property "Reference" "#PWR087"
+		(property "Reference" "#PWR088"
 			(at 259.08 161.29 0)
 			(effects
@@
 			(project "Lark"
 				(path "/a351af57-4353-47da-9f45-7393de572768/4f6e6a31-1617-4951-bb1f-ffce39c005db"
-					(reference "#PWR087")
+					(reference "#PWR088")
 					(unit 1)
 				)
@@
 		(dnp no)
 		(fields_autoplaced yes)
-		(property "Reference" "#PWR089"
+		(property "Reference" "#PWR090"
 			(at 24.13 170.18 0)
 			(effects
@@
 			(project "Lark"
 				(path "/a351af57-4353-47da-9f45-7393de572768/4f6e6a31-1617-4951-bb1f-ffce39c005db"
-					(reference "#PWR089")
+					(reference "#PWR090")
 					(unit 1)
 				)
@@
 		(dnp no)
 		(fields_autoplaced yes)
-		(property "Reference" "#PWR095"
+		(property "Reference" "#PWR096"
 			(at 85.09 191.77 0)
 			(effects
@@
 			(project "Lark"
 				(path "/a351af57-4353-47da-9f45-7393de572768/4f6e6a31-1617-4951-bb1f-ffce39c005db"
-					(reference "#PWR095")
+					(reference "#PWR096")
 					(unit 1)
 				)
@@
 		(dnp no)
 		(fields_autoplaced yes)
-		(property "Reference" "#PWR090"
+		(property "Reference" "#PWR091"
 			(at 53.34 170.18 0)
 			(effects
@@
 			(project "Lark"
 				(path "/a351af57-4353-47da-9f45-7393de572768/4f6e6a31-1617-4951-bb1f-ffce39c005db"
-					(reference "#PWR090")
+					(reference "#PWR091")
 					(unit 1)
 				)
@@
 		(dnp no)
 		(fields_autoplaced yes)
-		(property "Reference" "#PWR082"
+		(property "Reference" "#PWR083"
 			(at 270.51 104.14 0)
 			(effects
@@
 			(project "Lark"
 				(path "/a351af57-4353-47da-9f45-7393de572768/4f6e6a31-1617-4951-bb1f-ffce39c005db"
-					(reference "#PWR082")
+					(reference "#PWR083")
 					(unit 1)
 				)
@@
 		(dnp no)
 		(fields_autoplaced yes)
-		(property "Reference" "#PWR094"
+		(property "Reference" "#PWR095"
 			(at 53.34 191.77 0)
 			(effects
@@
 			(project "Lark"
 				(path "/a351af57-4353-47da-9f45-7393de572768/4f6e6a31-1617-4951-bb1f-ffce39c005db"
-					(reference "#PWR094")
+					(reference "#PWR095")
 					(unit 1)
 				)
@@
 		(on_board yes)
 		(dnp no)
-		(property "Reference" "C20"
+		(property "Reference" "C21"
 			(at 26.67 173.9962 0)
 			(effects
@@
 			(project "Lark"
 				(path "/a351af57-4353-47da-9f45-7393de572768/4f6e6a31-1617-4951-bb1f-ffce39c005db"
-					(reference "C20")
+					(reference "C21")
 					(unit 1)
 				)
@@
 		(dnp no)
 		(fields_autoplaced yes)
-		(property "Reference" "#PWR091"
+		(property "Reference" "#PWR092"
 			(at 85.09 170.18 0)
 			(effects
@@
 			(project "Lark"
 				(path "/a351af57-4353-47da-9f45-7393de572768/4f6e6a31-1617-4951-bb1f-ffce39c005db"
-					(reference "#PWR091")
+					(reference "#PWR092")
 					(unit 1)
 				)
@@
 		(dnp no)
 		(fields_autoplaced yes)
-		(property "Reference" "#PWR093"
+		(property "Reference" "#PWR094"
 			(at 38.1 191.77 0)
 			(effects
@@
 			(project "Lark"
 				(path "/a351af57-4353-47da-9f45-7393de572768/4f6e6a31-1617-4951-bb1f-ffce39c005db"
-					(reference "#PWR093")
+					(reference "#PWR094")
 					(unit 1)
 				)
@@
 		(dnp no)
 		(fields_autoplaced yes)
-		(property "Reference" "#PWR092"
+		(property "Reference" "#PWR093"
 			(at 24.13 191.77 0)
 			(effects
@@
 			(project "Lark"
 				(path "/a351af57-4353-47da-9f45-7393de572768/4f6e6a31-1617-4951-bb1f-ffce39c005db"
-					(reference "#PWR092")
+					(reference "#PWR093")
 					(unit 1)
 				)
@@
 		(dnp no)
 		(fields_autoplaced yes)
-		(property "Reference" "#PWR083"
+		(property "Reference" "#PWR084"
 			(at 163.83 119.38 0)
 			(effects
@@
 			(project "Lark"
 				(path "/a351af57-4353-47da-9f45-7393de572768/4f6e6a31-1617-4951-bb1f-ffce39c005db"
-					(reference "#PWR083")
+					(reference "#PWR084")
 					(unit 1)
 				)
@@
 		(on_board yes)
 		(dnp no)
-		(property "Reference" "C18"
+		(property "Reference" "C19"
 			(at 273.05 107.9562 0)
 			(effects
@@
 			(project "Lark"
 				(path "/a351af57-4353-47da-9f45-7393de572768/4f6e6a31-1617-4951-bb1f-ffce39c005db"
-					(reference "C18")
+					(reference "C19")
 					(unit 1)
 				)
@@
 		(on_board yes)
 		(dnp no)
-		(property "Reference" "U8"
+		(property "Reference" "U10"
 			(at 136.906 68.072 0)
 			(effects
@@
 			(project "Lark"
 				(path "/a351af57-4353-47da-9f45-7393de572768/4f6e6a31-1617-4951-bb1f-ffce39c005db"
-					(reference "U8")
+					(reference "U10")
 					(unit 1)
 				)
@@
 		(dnp no)
 		(fields_autoplaced yes)
-		(property "Reference" "#PWR088"
+		(property "Reference" "#PWR089"
 			(at 270.51 161.29 0)
 			(effects
@@
 			(project "Lark"
 				(path "/a351af57-4353-47da-9f45-7393de572768/4f6e6a31-1617-4951-bb1f-ffce39c005db"
-					(reference "#PWR088")
+					(reference "#PWR089")
 					(unit 1)
 				)
@@
 		(dnp no)
 		(fields_autoplaced yes)
-		(property "Reference" "#PWR079"
+		(property "Reference" "#PWR080"
 			(at 118.11 63.5 0)
 			(effects
@@
 			(project "Lark"
 				(path "/a351af57-4353-47da-9f45-7393de572768/4f6e6a31-1617-4951-bb1f-ffce39c005db"
-					(reference "#PWR079")
+					(reference "#PWR080")
 					(unit 1)
 				)
@@
 		(dnp no)
 		(fields_autoplaced yes)
-		(property "Reference" "#PWR085"
+		(property "Reference" "#PWR086"
 			(at 233.68 161.29 0)
 			(effects
@@
 			(project "Lark"
 				(path "/a351af57-4353-47da-9f45-7393de572768/4f6e6a31-1617-4951-bb1f-ffce39c005db"
-					(reference "#PWR085")
+					(reference "#PWR086")
 					(unit 1)
 				)
@@
 		(dnp no)
 		(fields_autoplaced yes)
-		(property "Reference" "#PWR084"
+		(property "Reference" "#PWR085"
 			(at 223.52 161.29 0)
 			(effects
@@
 			(project "Lark"
 				(path "/a351af57-4353-47da-9f45-7393de572768/4f6e6a31-1617-4951-bb1f-ffce39c005db"
-					(reference "#PWR084")
+					(reference "#PWR085")
 					(unit 1)
 				)
@@
 		(dnp no)
 		(fields_autoplaced yes)
-		(property "Reference" "#PWR086"
+		(property "Reference" "#PWR087"
 			(at 246.38 161.29 0)
 			(effects
@@
 			(project "Lark"
 				(path "/a351af57-4353-47da-9f45-7393de572768/4f6e6a31-1617-4951-bb1f-ffce39c005db"
-					(reference "#PWR086")
+					(reference "#PWR087")
 					(unit 1)
 				)
@@
 		(on_board yes)
 		(dnp no)
-		(property "Reference" "C17"
+		(property "Reference" "C18"
 			(at 260.35 107.9562 0)
 			(effects
@@
 			(project "Lark"
 				(path "/a351af57-4353-47da-9f45-7393de572768/4f6e6a31-1617-4951-bb1f-ffce39c005db"
-					(reference "C17")
+					(reference "C18")
 					(unit 1)
 				)
@@
 		(on_board yes)
 		(dnp no)
-		(property "Reference" "C21"
+		(property "Reference" "C22"
 			(at 40.64 173.9962 0)
 			(effects
@@
 			(project "Lark"
 				(path "/a351af57-4353-47da-9f45-7393de572768/4f6e6a31-1617-4951-bb1f-ffce39c005db"
-					(reference "C21")
+					(reference "C22")
 					(unit 1)
 				)
@@
 		(on_board yes)
 		(dnp no)
-		(property "Reference" "C22"
+		(property "Reference" "C23"
 			(at 55.88 173.9962 0)
 			(effects
@@
 			(project "Lark"
 				(path "/a351af57-4353-47da-9f45-7393de572768/4f6e6a31-1617-4951-bb1f-ffce39c005db"
-					(reference "C22")
-					(unit 1)
-				)
+					(reference "C23")
+					(unit 1)
+				)

Commit message: minor updates
- changed npn pins to passive.
- changed rev to match working revision.
- minor PCB changes.
- moved TVS diode next to connector.
- changed barrel jack silkscreen.
- changed usbc silkscreen.
Connections:
- net VERF renamed VREF
Changed lines of the file:
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@@
 		(title "Lark Print Engine")
 		(date "2025-10-08")
-		(rev "01.00.01")
+		(rev "01.00.00")
 		(comment 1 "Thermal Print Engine")
 		(comment 2 "Designer: HamSlices")
@@
 	(wire
 		(pts
-			(xy 26.67 143.51) (xy 20.32 143.51)
+			(xy 29.21 143.51) (xy 20.32 143.51)
 		)
 		(stroke
@@
 	)
 	(label "VREF"
-		(at 26.67 143.51 180)
+		(at 29.21 143.51 180)
 		(effects
 			(font
@@
 		)
 	)
-	(hierarchical_label "VERF"
+	(hierarchical_label "VREF"
 		(shape input)
 		(at 113.03 93.98 180)

Commit message: Changed revision again...
- It dawned on me that this is rev 2, so the rev is now 01.00.1.
- Added thermal relief to the TH pads so I can actually solder the parts.
- Added more silkscreen to denote the rev, the github link, and ESD sensitivity of the device.
- Made minor pcb changes, I moved a test point, and cleaned up some traces.
Parts:
- R36: value 100KΩ -> 100kΩ
- TP12: now left out of the parts list
