File: Lark/Resistor_Networks.kicad_sch (KiCad schematic)
At the start: 5 parts

Commit message: update, WIP
- Reannotated schematic.
- Added STM32 device.
- Fixed High-side switch (removed soft-start cap for device safety).
Parts:
- renumbered R31 to R44, RN3 to RN1, RN4 to RN3, RN1 to RN4
Changed lines of the file:
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@@
 		(dnp no)
 		(fields_autoplaced yes)
-		(property "Reference" "#PWR083"
+		(property "Reference" "#PWR0131"
 			(at 118.11 64.77 0)
 			(effects
@@
 			(project "Lark"
 				(path "/a351af57-4353-47da-9f45-7393de572768/6e291d34-e508-4d3b-a2e9-20acfef2b928/b7401ced-a663-484b-a6a1-a8142de0403d"
-					(reference "#PWR083")
+					(reference "#PWR0131")
 					(unit 1)
 				)
@@
 		(on_board yes)
 		(dnp no)
-		(property "Reference" "RN3"
+		(property "Reference" "RN1"
 			(at 129.54 73.152 0)
 			(effects
@@
 			(project "Lark"
 				(path "/a351af57-4353-47da-9f45-7393de572768/6e291d34-e508-4d3b-a2e9-20acfef2b928/b7401ced-a663-484b-a6a1-a8142de0403d"
-					(reference "RN3")
+					(reference "RN1")
 					(unit 1)
 				)
@@
 		(on_board yes)
 		(dnp no)
-		(property "Reference" "RN1"
+		(property "Reference" "RN4"
 			(at 173.99 106.934 90)
 			(effects
@@
 			(project "Lark"
 				(path "/a351af57-4353-47da-9f45-7393de572768/6e291d34-e508-4d3b-a2e9-20acfef2b928/b7401ced-a663-484b-a6a1-a8142de0403d"
-					(reference "RN1")
+					(reference "RN4")
 					(unit 1)
 				)
@@
 		(on_board yes)
 		(dnp no)
-		(property "Reference" "RN4"
+		(property "Reference" "RN3"
 			(at 173.99 91.694 90)
 			(effects
@@
 			(project "Lark"
 				(path "/a351af57-4353-47da-9f45-7393de572768/6e291d34-e508-4d3b-a2e9-20acfef2b928/b7401ced-a663-484b-a6a1-a8142de0403d"
-					(reference "RN4")
+					(reference "RN3")
 					(unit 1)
 				)
@@
 		(on_board yes)
 		(dnp no)
-		(property "Reference" "R31"
+		(property "Reference" "R44"
 			(at 171.704 123.19 90)
 			(effects
@@
 			(project "Lark"
 				(path "/a351af57-4353-47da-9f45-7393de572768/6e291d34-e508-4d3b-a2e9-20acfef2b928/b7401ced-a663-484b-a6a1-a8142de0403d"
-					(reference "R31")
+					(reference "R44")
 					(unit 1)
 				)
@@
 		(dnp no)
 		(fields_autoplaced yes)
-		(property "Reference" "#PWR084"
+		(property "Reference" "#PWR0132"
 			(at 137.16 64.77 0)
 			(effects
@@
 			(project "Lark"
 				(path "/a351af57-4353-47da-9f45-7393de572768/6e291d34-e508-4d3b-a2e9-20acfef2b928/b7401ced-a663-484b-a6a1-a8142de0403d"
-					(reference "#PWR084")
-					(unit 1)
-				)
+					(reference "#PWR0132")
+					(unit 1)
+				)

Commit message: Updated schematic, WIP
- Added NOR flash part.
- Added new CubeMX config file.
- Reannotated the schematic.
- Made some more connections to the MCU.
Parts:
- renumbered R44 to R45
Changed lines of the file:
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@@
 		(on_board yes)
 		(dnp no)
-		(property "Reference" "R44"
+		(property "Reference" "R45"
 			(at 171.704 123.19 90)
 			(effects
@@
 			(project "Lark"
 				(path "/a351af57-4353-47da-9f45-7393de572768/6e291d34-e508-4d3b-a2e9-20acfef2b928/b7401ced-a663-484b-a6a1-a8142de0403d"
-					(reference "R44")
+					(reference "R45")
 					(unit 1)
 				)

Commit message: Update, WIP
- Added TVS diode to 24v Supply.
- Fixed bleeder circuit at some point (I think it was this commit)
- Added Jumper to connect NTC to ADC. (again I think it was this commit)
Parts:
- renumbered R45 to R48
Changed lines of the file:
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@@
 		(dnp no)
 		(fields_autoplaced yes)
-		(property "Reference" "#PWR0131"
+		(property "Reference" "#PWR0135"
 			(at 118.11 64.77 0)
 			(effects
@@
 			(project "Lark"
 				(path "/a351af57-4353-47da-9f45-7393de572768/6e291d34-e508-4d3b-a2e9-20acfef2b928/b7401ced-a663-484b-a6a1-a8142de0403d"
-					(reference "#PWR0131")
+					(reference "#PWR0135")
 					(unit 1)
 				)
@@
 		(on_board yes)
 		(dnp no)
-		(property "Reference" "R45"
+		(property "Reference" "R48"
 			(at 171.704 123.19 90)
 			(effects
@@
 			(project "Lark"
 				(path "/a351af57-4353-47da-9f45-7393de572768/6e291d34-e508-4d3b-a2e9-20acfef2b928/b7401ced-a663-484b-a6a1-a8142de0403d"
-					(reference "R45")
+					(reference "R48")
 					(unit 1)
 				)
@@
 		(dnp no)
 		(fields_autoplaced yes)
-		(property "Reference" "#PWR0132"
+		(property "Reference" "#PWR0136"
 			(at 137.16 64.77 0)
 			(effects
@@
 			(project "Lark"
 				(path "/a351af57-4353-47da-9f45-7393de572768/6e291d34-e508-4d3b-a2e9-20acfef2b928/b7401ced-a663-484b-a6a1-a8142de0403d"
-					(reference "#PWR0132")
-					(unit 1)
-				)
+					(reference "#PWR0136")
+					(unit 1)
+				)

Commit message: started on layout, WIP
I'm not a fan of how its going, I feel like I might redo it, before I get to far into it. A patchy foundation makes an unstable house.
Connections:
- net N1: now also RN1.4 (R4.1); no longer RN1.1 (R1.1)
- net N2: now also RN1.3 (R3.1); no longer RN1.2 (R2.1)
- net N3: now also RN1.2 (R2.1); no longer RN1.3 (R3.1)
- net N4: now also RN1.1 (R1.1); no longer RN1.4 (R4.1)
- net N5: now also RN2.4 (R4.1); no longer RN2.1 (R1.1)
- net N7: now also RN2.1 (R1.1)
- net N9: no longer RN2.4 (R4.1)
Other:
- note added: "No Pullup"
