File: Kicad Project Files/STLink_adapter/Adapter.kicad_sch (KiCad schematic)
At the start: 2 parts, among them J1 0530470410, J2 SFH11-PBPC-D10-ST-BK

Commit message: Added gerbers + bill of materials
- Changed connector symbol to include MPN.
- Added DNP field to lark BOM
Parts:
- J2: MPN (none) -> SFH11-PBPC-D10-ST-BK
Changed lines of the file:
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@@
+			)
+		)
+		(property "MPN" "SFH11-PBPC-D10-ST-BK"
+			(at 22.86 72.39 0)
+			(effects
+				(font
+					(size 1.27 1.27)
+				)
+				(hide yes)
 			)
 		)
