File: Kicad Project Files/Lark/Auxiliary.kicad_sch (KiCad schematic)
At the start: 9 parts, among them J6 0530470210, J7 0530470410, J8 0530470410

Commit message: Added Notes
- Changed AUX power to FAN power, added note about fan.
- Changed bottom and top silk.
- Added 24v pour to the top of connector j4, the mid 24v pins remain the same.
Other:
- note added: "- Recomended Fan - Sunon Fans MF50152V1-1000U-A99 50mm x 50mm x 15.00mm 24V, 1.01 Watts"
- note added: "FAN 24V Power"
- note removed: "AUX 24V Power"
Changed lines of the file:
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@@
+	)
+	(rectangle
+		(start 254 58.166)
+		(end 278.13 71.12)
+		(stroke
+			(width 0)
+			(type dash)
+		)
+		(fill
+			(type none)
+		)
 	)
 	(rectangle
@@
 		)
 	)
-	(text "AUX 24V Power"
+	(text "FAN 24V Power"
 		(exclude_from_sim no)
 		(at 253.746 17.78 0)
@@
 			)
 		)
+	)
+	(text "- Recomended Fan -\nSunon Fans\nMF50152V1-1000U-A99\n50mm x 50mm x 15.00mm\n24V, 1.01 Watts"
+		(exclude_from_sim no)
+		(at 266.192 64.516 0)
+		(effects
+			(font
+				(face "Consolas")
+				(size 1.27 1.27)
+			)
+		)
