File: Kicad Project Files/FrontIO/FrontIO.kicad_pcb (KiCad board)
At the start: 2 copper layers, 86 x 14 mm, 8 parts, among them J1 0530470810, J2 0530470210, SW1 TS04-66-65-BK-100-SMT, SW2 TS04-66-65-BK-100-SMT, SW3 TS04-66-65-BK-100-SMT

Commit message: updated broken QR on Front IO PCB and SCH.
Parts:
- moved G*** 0.70 mm to (127.1, 97.2)
